File: project/SchedaRobotica.brd (EAGLE design)
At the start: 210 x 210 mm, 115 parts, among them IC1 LMZ14202TZE-ADJ_NOPB, IC2 VNH7070ASTR, IC3 VNH7070ASTR, IC4 VNH7070ASTR, IC5 VNH7070ASTR, M1 43650-0201, M2 43650-0201, M3 43650-0201, M4 43650-0201

Commit message: mh, kinda dunno what to do
Parts:
- removed B_SW_1, B_SW_2: 21810LPSTF, 21810LPSTF:SOIC127P844X265-20N
- moved SV6 287.2 mm to (81.3, -5.08), turned to 90 degrees
- moved SV2 2.54 mm to (-20.2, 71.5)
- turned S3 to 140 degrees
Connections:
- net B1: now also ARDUINO1.A2, SV2.3, SV6.8, U$1.10-CS\MQSR
- net B2: now also ARDUINO1.A1, SV2.4, SV6.9, U$1.11-MOSI/CTX1
Changed lines of the file:
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@@
 <attribute name="NAME" x="25.6844" y="93.966265625" size="1.27" layer="26" ratio="10" rot="MR200"/>
 </element>
-<element name="S3" library="adafruit" package="PNA460XM" value="PNA460XM" x="-59.718525" y="80.1517" smashed="yes" rot="MR145">
-<attribute name="NAME" x="-61.852959375" y="76.42461875" size="1.27" layer="26" ratio="10" rot="MR145"/>
+<element name="S3" library="adafruit" package="PNA460XM" value="PNA460XM" x="-59.718525" y="80.1517" smashed="yes" rot="MR140">
+<attribute name="NAME" x="-61.52" y="76.252771875" size="1.27" layer="26" ratio="10" rot="MR140"/>
 </element>
 <element name="S4" library="adafruit" package="PNA460XM" value="PNA460XM" x="-81.8417" y="58.028525" smashed="yes" rot="MR125">
@@
 <attribute name="VALUE" x="15.477" y="68.609" size="1.27" layer="27" ratio="10"/>
 </element>
-<element name="SV2" library="con-lstb" library_urn="urn:adsk.eagle:library:162" package="MA12-1" package3d_urn="urn:adsk.eagle:package:8348/1" value="" x="-17.67" y="71.53" smashed="yes">
-<attribute name="MF" value="" x="43.29" y="11.84" size="1.778" layer="27" display="off"/>
-<attribute name="MPN" value="" x="43.29" y="11.84" size="1.778" layer="27" display="off"/>
-<attribute name="NAME" x="-32.91" y="73.308" size="1.27" layer="25" ratio="10"/>
-<attribute name="OC_FARNELL" value="unknown" x="43.29" y="11.84" size="1.778" layer="27" display="off"/>
-<attribute name="OC_NEWARK" value="unknown" x="43.29" y="11.84" size="1.778" layer="27" display="off"/>
-<attribute name="POPULARITY" value="2" x="43.29" y="11.84" size="1.778" layer="27" display="off"/>
-<attribute name="VALUE" x="-16.273" y="68.609" size="1.27" layer="27" ratio="10"/>
+<element name="SV2" library="con-lstb" library_urn="urn:adsk.eagle:library:162" package="MA12-1" package3d_urn="urn:adsk.eagle:package:8348/1" value="" x="-20.21" y="71.53" smashed="yes">
+<attribute name="MF" value="" x="40.75" y="11.84" size="1.778" layer="27" display="off"/>
+<attribute name="MPN" value="" x="40.75" y="11.84" size="1.778" layer="27" display="off"/>
+<attribute name="NAME" x="-35.45" y="73.308" size="1.27" layer="25" ratio="10"/>
+<attribute name="OC_FARNELL" value="unknown" x="40.75" y="11.84" size="1.778" layer="27" display="off"/>
+<attribute name="OC_NEWARK" value="unknown" x="40.75" y="11.84" size="1.778" layer="27" display="off"/>
+<attribute name="POPULARITY" value="2" x="40.75" y="11.84" size="1.778" layer="27" display="off"/>
+<attribute name="VALUE" x="-18.813" y="68.609" size="1.27" layer="27" ratio="10"/>
 </element>
 <element name="SV3" library="con-lstb" library_urn="urn:adsk.eagle:library:162" package="MA12-1" package3d_urn="urn:adsk.eagle:package:8348/1" value="" x="-18.94" y="41.05" smashed="yes">
@@
 <attribute name="VALUE" x="-171.323" y="-107.061" size="1.27" layer="27" ratio="10"/>
 </element>
-<element name="SV6" library="SparkFun-Connectors" package="1X14-LONGPADS" value="" x="-185.42" y="-111.76" smashed="yes">
-<attribute name="NAME" x="-186.69" y="-110.363" size="0.6096" layer="25" font="vector" ratio="20"/>
-<attribute name="VALUE" x="-186.69" y="-113.792" size="0.6096" layer="27" font="vector" ratio="20"/>
-</element>
-<element name="B_SW_1" library="21810LPSTF" package="SOIC127P844X265-20N" value="21810LPSTF" x="44.45" y="-43.18" smashed="yes" rot="R270">
-<attribute name="DESCRIPTION" value="DIP SW,Half-pitch,10-pos,flush act,SMD" x="44.45" y="-43.18" size="1.778" layer="27" rot="R270" display="off"/>
-<attribute name="HEIGHT" value="2.65mm" x="44.45" y="-43.18" size="1.778" layer="27" rot="R270" display="off"/>
-<attribute name="MANUFACTURER_NAME" value="CTS" x="44.45" y="-43.18" size="1.778" layer="27" rot="R270" display="off"/>
-<attribute name="MANUFACTURER_PART_NUMBER" value="21810LPSTF" x="44.45" y="-43.18" size="1.778" layer="27" rot="R270" display="off"/>
-<attribute name="NAME" x="44.45" y="-49.53" size="1.27" layer="25" align="center"/>
-<attribute name="RS_PART_NUMBER" value="" x="44.45" y="-43.18" size="1.778" layer="27" rot="R270" display="off"/>
-<attribute name="RS_PRICE-STOCK" value="" x="44.45" y="-43.18" size="1.778" layer="27" rot="R270" display="off"/>
-<attribute name="VALUE" x="44.45" y="-43.18" size="1.27" layer="27" rot="R270" align="center"/>
-</element>
-<element name="B_SW_2" library="21810LPSTF" package="SOIC127P844X265-20N" value="21810LPSTF" x="59.69" y="-43.18" smashed="yes" rot="R270">
-<attribute name="DESCRIPTION" value="DIP SW,Half-pitch,10-pos,flush act,SMD" x="74.93" y="-30.48" size="1.778" layer="27" rot="R270" display="off"/>
-<attribute name="HEIGHT" value="2.65mm" x="74.93" y="-30.48" size="1.778" layer="27" rot="R270" display="off"/>
-<attribute name="MANUFACTURER_NAME" value="CTS" x="74.93" y="-30.48" size="1.778" layer="27" rot="R270" display="off"/>
-<attribute name="MANUFACTURER_PART_NUMBER" value="21810LPSTF" x="74.93" y="-30.48" size="1.778" layer="27" rot="R270" display="off"/>
-<attribute name="NAME" x="59.69" y="-49.53" size="1.27" layer="25" align="center"/>
-<attribute name="RS_PART_NUMBER" value="" x="74.93" y="-30.48" size="1.778" layer="27" rot="R270" display="off"/>
-<attribute name="RS_PRICE-STOCK" value="" x="74.93" y="-30.48" size="1.778" layer="27" rot="R270" display="off"/>
-<attribute name="VALUE" x="59.69" y="-43.18" size="1.27" layer="27" rot="R270" align="center"/>
+<element name="SV6" library="SparkFun-Connectors" package="1X14-LONGPADS" value="" x="81.28" y="-5.08" smashed="yes" rot="R90">
+<attribute name="NAME" x="79.883" y="-6.35" size="0.6096" layer="25" font="vector" ratio="20" rot="R90"/>
+<attribute name="VALUE" x="83.312" y="-6.35" size="0.6096" layer="27" font="vector" ratio="20" rot="R90"/>
 </element>
 </elements>
@@
 <wire x1="-144.35" y1="6.35" x2="-129.13" y2="-56.09" width="0" layer="19" extent="1-1"/>
 <wire x1="-80.38481875" y1="60.10916875" x2="-144.35" y2="6.35" width="0" layer="19" extent="1-1"/>
-<wire x1="-61.799171875" y1="78.694815625" x2="-80.38481875" y2="60.10916875" width="0" layer="19" extent="1-1"/>
-<wire x1="-29.45488125" y1="95.22438125" x2="-61.799171875" y2="78.694815625" width="0" layer="19" extent="1-1"/>
+<wire x1="-61.664278125" y1="78.51901875" x2="-80.38481875" y2="60.10916875" width="0" layer="19" extent="1-1"/>
+<wire x1="-29.45488125" y1="95.22438125" x2="-61.664278125" y2="78.51901875" width="0" layer="19" extent="1-1"/>
 <wire x1="-3.48" y1="99.25" x2="-29.45488125" y2="95.22438125" width="0" layer="19" extent="1-1"/>
 </signal>
 <signal name="B1">
 <contactref element="S1" pad="3"/>
+<contactref element="U$1" pad="10-CS\MQSR"/>
+<contactref element="SV2" pad="3"/>
+<contactref element="ARDUINO1" pad="A2"/>
+<contactref element="SV6" pad="8"/>
+<wire x1="-29.1" y1="71.53" x2="1.6" y2="99.25" width="0" layer="19" extent="1-1"/>
+<wire x1="-2.43" y1="48.67" x2="-29.1" y2="71.53" width="0" layer="19" extent="1-1"/>
+<wire x1="71.23" y1="10.57" x2="-2.43" y2="48.67" width="0" layer="19" extent="1-1"/>
+<wire x1="81.28" y1="12.7" x2="71.23" y2="10.57" width="0" layer="19" extent="1-1"/>
 </signal>
 <signal name="B2">
 <contactref element="S2" pad="1"/>
+<contactref element="U$1" pad="11-MOSI/CTX1"/>
+<contactref element="SV2" pad="4"/>
+<contactref element="ARDUINO1" pad="A1"/>
+<contactref element="SV6" pad="9"/>
+<wire x1="0.11" y1="48.67" x2="71.23" y2="8.03" width="0" layer="19" extent="1-1"/>
+<wire x1="-26.56" y1="71.53" x2="0.11" y2="48.67" width="0" layer="19" extent="1-1"/>
+<wire x1="-34.228521875" y1="93.486921875" x2="-26.56" y2="71.53" width="0" layer="19" extent="1-1"/>
+<wire x1="81.28" y1="15.24" x2="0.11" y2="48.67" width="0" layer="19" extent="1-1"/>
 </signal>
 <signal name="B3">

Commit message: mh, kinda dunno what to do part. 2
Parts:
- added SV10, SV11, SV12, SV13, SV14, SV15, SV16, SV7, SV8, SV9: (no value), con-lstb:MA03-1
- moved C2 398.8 mm to (20.3, -69.8), turned to 90 degrees
- moved C3 395.0 mm to (22.9, -69.8), turned to 90 degrees
- moved IC1 392.0 mm to (19.1, -63.5)
- moved C8 388.4 mm to (31.8, -64.0), turned to 90 degrees
- moved C5 384.3 mm to (34.3, -63.5), turned to 90 degrees
- moved C6 380.7 mm to (36.8, -63.5), turned to 90 degrees
- moved C1 357.0 mm to (20.3, -26.7)
- moved C7 343.0 mm to (20.3, -41.9)
- moved C4 329.4 mm to (7.62, -39.4)
- moved C9 329.4 mm to (7.62, -45.7)
- moved R1 329.4 mm to (7.62, -52.1)
- moved R2 329.4 mm to (7.62, -57.1)
- moved R3 329.4 mm to (7.62, -62.2)
- moved SV5 254.3 mm to (66.0, -16.5)
- moved C10 253.5 mm to (33.0, -11.4), turned to 180 degrees
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
Commit message: mh, kinda dunno what to do part. 3, but added supply and arranged things
Parts:
- R1: value (none) -> 61,9k
- R2: value (none) -> 1,07k
- R3: value (none) -> 3,32k
- SW_ELETT, SW_MOT: device switch:255SB -> switch_modified:255SB
- moved SV13 148.4 mm to (-96.5, -0.76), turned to 90 degrees
- moved R11 145.1 mm to (-45.7, -1.27)
- moved R9 145.1 mm to (-40.6, -1.27)
- moved M3+ 136.1 mm to (-55.1, -15.5), turned to 90 degrees
- moved M3- 133.5 mm to (-55.1, -17.8), turned to 90 degrees
- moved R12 128.5 mm to (-47.0, 35.6)
- moved C18 123.7 mm to (-62.2, -26.7)
- moved R17 123.7 mm to (-57.1, -26.7)
- moved R18 123.7 mm to (-52.1, -26.7)
- moved R19 123.7 mm to (-62.2, -31.8)
- moved R20 123.7 mm to (-57.1, -31.8)
- moved SV16 123.6 mm to (-0.76, -96.3), turned to 180 degrees
- moved R13 122.5 mm to (-63.5, 50.8)
- moved R16 122.5 mm to (-63.5, 45.7)
- moved C16 122.5 mm to (-68.6, 50.8)
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- renumbered IC2 to DRV1, IC3 to DRV3, IC4 to DRV2, IC5 to DRV4
Other:
- board size 210 x 210 mm -> 228.6 x 231.1 mm

Commit message: part 3
Parts:
- removed ARDUINO1: (no value), arduinopromini:ARDUINO_PRO_MINI
- added SV17, SV18, SV19, SV20, SV21, SV22, SV23, SV24, SV25, SV26: (no value), con-lstb:MA03-1
Connections:
- removed net VCC: ARDUINO1.VCC, ARDUINO1.VCC@1
- net B1: no longer ARDUINO1.A2
- net B2: no longer ARDUINO1.A1
- net GND: no longer ARDUINO1.GND, ARDUINO1.GND@1, ARDUINO1.GND@2, ARDUINO1.GND@3
