File: project/SchedaRobotica.sch (EAGLE design)
At the start: 115 parts, among them IC1 LMZ14202TZE-ADJ_NOPB, IC2 VNH7070ASTR, IC3 VNH7070ASTR, IC4 VNH7070ASTR, IC5 VNH7070ASTR, M1 43650-0201, M2 43650-0201, M3 43650-0201, M4 43650-0201

Commit message: mh, kinda dunno what to do
Parts:
- removed B_SW_1, B_SW_2: 21810LPSTF, 21810LPSTF:21810LPSTF
Connections:
- net B1: now also ARDUINO1.A2, SV2.3, SV6.8, U$1.10-CS/MQSR
- net B2: now also ARDUINO1.A1, SV2.4, SV6.9, U$1.11-MOSI/CTX1
Other:
- moved on the sheet: SV6
Changed lines of the file:
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@@
 <setting verticaltext="up"/>
 </settings>
-<grid distance="0.1" unitdist="inch" unit="inch" style="dots" multiple="1" display="yes" altdistance="0.05" altunitdist="inch" altunit="inch"/>
+<grid distance="0.1" unitdist="inch" unit="inch" style="dots" multiple="1" display="yes" altdistance="0.01" altunitdist="inch" altunit="inch"/>
 <layers>
 <layer number="1" name="Top" color="4" fill="1" visible="no" active="no"/>
@@
 <part name="SV5" library="con-lstb" library_urn="urn:adsk.eagle:library:162" deviceset="MA12-1" device="" package3d_urn="urn:adsk.eagle:package:8348/1"/>
 <part name="SV6" library="SparkFun-Connectors" deviceset="CONN_14" device="LONGPADS"/>
-<part name="B_SW_1" library="21810LPSTF" deviceset="21810LPSTF" device=""/>
-<part name="B_SW_2" library="21810LPSTF" deviceset="21810LPSTF" device=""/>
 </parts>
 <sheets>
@@
 <wire x1="271.78" y1="185.42" x2="220.98" y2="185.42" width="0.1524" layer="97"/>
 <text x="220.98" y="139.7" size="1.778" layer="97">MOTOR CONS</text>
-<text x="345.44" y="304.8" size="1.778" layer="91">TODO:
+<text x="325.12" y="157.48" size="1.778" layer="91">TODO:
 -add serials and values
 -add roller and kicker connectors (?)
@@
 <attribute name="NAME" x="120.65" y="97.282" size="1.778" layer="95"/>
 </instance>
-<instance part="SV6" gate="G$1" x="182.88" y="55.88" smashed="yes" rot="R180">
-<attribute name="VALUE" x="182.88" y="78.486" size="1.778" layer="96" font="vector" rot="R180"/>
-<attribute name="NAME" x="182.88" y="37.592" size="1.778" layer="95" font="vector" rot="R180"/>
-</instance>
-<instance part="B_SW_1" gate="G$1" x="350.52" y="223.52" smashed="yes">
-<attribute name="NAME" x="356.87" y="228.6" size="1.778" layer="95" align="center-left"/>
-</instance>
-<instance part="B_SW_2" gate="G$1" x="386.08" y="223.52" smashed="yes">
-<attribute name="NAME" x="392.43" y="228.6" size="1.778" layer="95" align="center-left"/>
+<instance part="SV6" gate="G$1" x="185.42" y="76.2" smashed="yes" rot="R180">
+<attribute name="VALUE" x="185.42" y="98.806" size="1.778" layer="96" font="vector" rot="R180"/>
+<attribute name="NAME" x="185.42" y="57.912" size="1.778" layer="95" font="vector" rot="R180"/>
 </instance>
 </instances>
@@
 <label x="317.5" y="30.48" size="1.778" layer="95"/>
 </segment>
+<segment>
+<pinref part="U$1" gate="G$1" pin="10-CS/MQSR"/>
+<pinref part="SV2" gate="1" pin="3"/>
+<wire x1="68.58" y1="48.26" x2="78.74" y2="48.26" width="0.1524" layer="91"/>
+<label x="68.58" y="48.26" size="1.778" layer="95"/>
+</segment>
+<segment>
+<pinref part="ARDUINO1" gate="G$1" pin="A2"/>
+<pinref part="SV6" gate="G$1" pin="8"/>
+<wire x1="165.1" y1="76.2" x2="175.26" y2="76.2" width="0.1524" layer="91"/>
+<label x="165.1" y="76.2" size="1.778" layer="95"/>
+</segment>
 </net>
 <net name="B2" class="0">
@@
 <label x="335.28" y="30.48" size="1.778" layer="95"/>
 </segment>
+<segment>
+<pinref part="U$1" gate="G$1" pin="11-MOSI/CTX1"/>
+<pinref part="SV2" gate="1" pin="4"/>
+<wire x1="68.58" y1="45.72" x2="78.74" y2="45.72" width="0.1524" layer="91"/>
+<label x="68.58" y="45.72" size="1.778" layer="95"/>
+</segment>
+<segment>
+<pinref part="ARDUINO1" gate="G$1" pin="A1"/>
+<pinref part="SV6" gate="G$1" pin="9"/>
+<wire x1="165.1" y1="73.66" x2="175.26" y2="73.66" width="0.1524" layer="91"/>
+<label x="167.64" y="73.66" size="1.778" layer="95"/>
+</segment>
 </net>

Commit message: mh, kinda dunno what to do part. 2
Parts:
- added SV10, SV11, SV12, SV13, SV14, SV15, SV16, SV7, SV8, SV9: (no value), con-lstb:MA03-1
Other:
- note added: "BALL PINHEADERS"
- note removed: "BALL SWITCHES"
Changed lines of the file:
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@@
 <part name="SV5" library="con-lstb" library_urn="urn:adsk.eagle:library:162" deviceset="MA12-1" device="" package3d_urn="urn:adsk.eagle:package:8348/1"/>
 <part name="SV6" library="SparkFun-Connectors" deviceset="CONN_14" device="LONGPADS"/>
+<part name="SV7" library="con-lstb" library_urn="urn:adsk.eagle:library:162" deviceset="MA03-1" device="" package3d_urn="urn:adsk.eagle:package:8339/1"/>
+<part name="SV8" library="con-lstb" library_urn="urn:adsk.eagle:library:162" deviceset="MA03-1" device="" package3d_urn="urn:adsk.eagle:package:8339/1"/>
+<part name="SV9" library="con-lstb" library_urn="urn:adsk.eagle:library:162" deviceset="MA03-1" device="" package3d_urn="urn:adsk.eagle:package:8339/1"/>
+<part name="SV10" library="con-lstb" library_urn="urn:adsk.eagle:library:162" deviceset="MA03-1" device="" package3d_urn="urn:adsk.eagle:package:8339/1"/>
+<part name="SV11" library="con-lstb" library_urn="urn:adsk.eagle:library:162" deviceset="MA03-1" device="" package3d_urn="urn:adsk.eagle:package:8339/1"/>
+<part name="SV12" library="con-lstb" library_urn="urn:adsk.eagle:library:162" deviceset="MA03-1" device="" package3d_urn="urn:adsk.eagle:package:8339/1"/>
+<part name="SV13" library="con-lstb" library_urn="urn:adsk.eagle:library:162" deviceset="MA03-1" device="" package3d_urn="urn:adsk.eagle:package:8339/1"/>
+<part name="SV14" library="con-lstb" library_urn="urn:adsk.eagle:library:162" deviceset="MA03-1" device="" package3d_urn="urn:adsk.eagle:package:8339/1"/>
+<part name="SV15" library="con-lstb" library_urn="urn:adsk.eagle:library:162" deviceset="MA03-1" device="" package3d_urn="urn:adsk.eagle:package:8339/1"/>
+<part name="SV16" library="con-lstb" library_urn="urn:adsk.eagle:library:162" deviceset="MA03-1" device="" package3d_urn="urn:adsk.eagle:package:8339/1"/>
 </parts>
 <sheets>
@@
 <text x="492.76" y="76.2" size="1.778" layer="97">BLUETOOTH</text>
 <wire x1="332.74" y1="238.76" x2="332.74" y2="190.5" width="0.1524" layer="97"/>
-<wire x1="332.74" y1="190.5" x2="421.64" y2="190.5" width="0.1524" layer="97"/>
-<wire x1="421.64" y1="190.5" x2="421.64" y2="238.76" width="0.1524" layer="97"/>
-<wire x1="421.64" y1="238.76" x2="332.74" y2="238.76" width="0.1524" layer="97"/>
-<text x="332.74" y="187.96" size="1.778" layer="97">BALL SWITCHES</text>
+<wire x1="332.74" y1="190.5" x2="431.8" y2="190.5" width="0.1524" layer="97"/>
+<wire x1="431.8" y1="190.5" x2="431.8" y2="238.76" width="0.1524" layer="97"/>
+<wire x1="431.8" y1="238.76" x2="332.74" y2="238.76" width="0.1524" layer="97"/>
+<text x="332.74" y="187.96" size="1.778" layer="97">BALL PINHEADERS</text>
 </plain>
 <instances>
@@
 <attribute name="NAME" x="185.42" y="57.912" size="1.778" layer="95" font="vector" rot="R180"/>
 </instance>
+<instance part="SV7" gate="G$1" x="337.82" y="228.6" smashed="yes">
+<attribute name="VALUE" x="336.55" y="220.98" size="1.778" layer="96"/>
+<attribute name="NAME" x="336.55" y="234.442" size="1.778" layer="95"/>
+</instance>
+<instance part="SV8" gate="G$1" x="337.82" y="213.36" smashed="yes">
+<attribute name="VALUE" x="336.55" y="205.74" size="1.778" layer="96"/>
+<attribute name="NAME" x="336.55" y="219.202" size="1.778" layer="95"/>
+</instance>
+<instance part="SV9" gate="G$1" x="353.06" y="228.6" smashed="yes">
+<attribute name="VALUE" x="351.79" y="220.98" size="1.778" layer="96"/>
+<attribute name="NAME" x="351.79" y="234.442" size="1.778" layer="95"/>
+</instance>
+<instance part="SV10" gate="G$1" x="353.06" y="213.36" smashed="yes">
+<attribute name="VALUE" x="351.79" y="205.74" size="1.778" layer="96"/>
+<attribute name="NAME" x="351.79" y="219.202" size="1.778" layer="95"/>
+</instance>
+<instance part="SV11" gate="G$1" x="368.3" y="228.6" smashed="yes">
+<attribute name="VALUE" x="367.03" y="220.98" size="1.778" layer="96"/>
+<attribute name="NAME" x="367.03" y="234.442" size="1.778" layer="95"/>
+</instance>
+<instance part="SV12" gate="G$1" x="368.3" y="213.36" smashed="yes">
+<attribute name="VALUE" x="367.03" y="205.74" size="1.778" layer="96"/>
+<attribute name="NAME" x="367.03" y="219.202" size="1.778" layer="95"/>
+</instance>
+<instance part="SV13" gate="G$1" x="383.54" y="228.6" smashed="yes">
+<attribute name="VALUE" x="382.27" y="220.98" size="1.778" layer="96"/>
+<attribute name="NAME" x="382.27" y="234.442" size="1.778" layer="95"/>
+</instance>
+<instance part="SV14" gate="G$1" x="383.54" y="213.36" smashed="yes">
+<attribute name="VALUE" x="382.27" y="205.74" size="1.778" layer="96"/>
+<attribute name="NAME" x="382.27" y="219.202" size="1.778" layer="95"/>
+</instance>
+<instance part="SV15" gate="G$1" x="398.78" y="228.6" smashed="yes">
+<attribute name="VALUE" x="397.51" y="220.98" size="1.778" layer="96"/>
+<attribute name="NAME" x="397.51" y="234.442" size="1.778" layer="95"/>
+</instance>
+<instance part="SV16" gate="G$1" x="398.78" y="213.36" smashed="yes">
+<attribute name="VALUE" x="397.51" y="205.74" size="1.778" layer="96"/>
+<attribute name="NAME" x="397.51" y="219.202" size="1.778" layer="95"/>
+</instance>
 </instances>

Commit message: mh, kinda dunno what to do part. 3, but added supply and arranged things
Parts:
- R1: value (none) -> 61,9k
- R2: value (none) -> 1,07k
- R3: value (none) -> 3,32k
- SW_ELETT, SW_MOT: device switch:255SB -> switch_modified:255SB
- renumbered IC2 to DRV1, IC3 to DRV3, IC4 to DRV2, IC5 to DRV4
Other:
- note added: "TODO: -add serials and values -add roller and kicker connectors (?) -add US cons if there's room -decide which uc, arduino promini (16 sensors) or nano 33 BLE (cooler, allows for 20 sensors) -add mux!!!! NOTE: in brd the spacing of ball sensor is inconsistent in S3, S5, S13"
- note removed: "TODO: -add serials and values -add roller and kicker connectors (?) -add US cons if there's room NOTE: in brd the spacing of ball sensor is inconsistent in S3, S5, S13"

Commit message: part 3
Parts:
- removed ARDUINO1: (no value), arduinopromini:ARDUINO_PRO_MINI
- added SV17, SV18, SV19, SV20, SV21, SV22, SV23, SV24, SV25, SV26: (no value), con-lstb:MA03-1
Connections:
- net B1: no longer ARDUINO1.A2
- net B2: no longer ARDUINO1.A1
Other:
- note added: "TODO: -add serials and values -add mux!!!! NOTE: in brd the spacing of ball sensor is inconsistent in S3, S5, S13 TODO if i have space: -roller/kicker cons -US cons"
- note removed: "TODO: -add serials and values -add roller and kicker connectors (?) -add US cons if there's room -decide which uc, arduino promini (16 sensors) or nano 33 BLE (cooler, allows for 20 sensors) -add mux!!!! NOTE: in brd the spacing of ball sensor is inconsistent in S3, S5, S13"
Changed lines of the file:
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@@
 <setting verticaltext="up"/>
 </settings>
-<grid distance="0.1" unitdist="inch" unit="inch" style="lines" multiple="1" display="no" altdistance="0.01" altunitdist="inch" altunit="inch"/>
+<grid distance="0.1" unitdist="inch" unit="inch" style="dots" multiple="1" display="yes" altdistance="0.01" altunitdist="inch" altunit="inch"/>
 <layers>
 <layer number="1" name="Top" color="4" fill="1" visible="no" active="no"/>
@@
 <part name="SV3" library="con-lstb" library_urn="urn:adsk.eagle:library:162" deviceset="MA12-1" device="" package3d_urn="urn:adsk.eagle:package:8348/1"/>
 <part name="SV4" library="con-lstb" library_urn="urn:adsk.eagle:library:162" deviceset="MA12-1" device="" package3d_urn="urn:adsk.eagle:package:8348/1"/>
-<part name="ARDUINO1" library="arduinopromini" deviceset="ARDUINO_PRO_MINI" device=""/>
 <part name="S1" library="adafruit" deviceset="PNA460XM" device=""/>
 <part name="S3" library="adafruit" deviceset="PNA460XM" device=""/>
@@
 <part name="SV15" library="con-lstb" library_urn="urn:adsk.eagle:library:162" deviceset="MA03-1" device="" package3d_urn="urn:adsk.eagle:package:8339/1"/>
 <part name="SV16" library="con-lstb" library_urn="urn:adsk.eagle:library:162" deviceset="MA03-1" device="" package3d_urn="urn:adsk.eagle:package:8339/1"/>
+<part name="SV17" library="con-lstb" library_urn="urn:adsk.eagle:library:162" deviceset="MA03-1" device="" package3d_urn="urn:adsk.eagle:package:8339/1"/>
+<part name="SV18" library="con-lstb" library_urn="urn:adsk.eagle:library:162" deviceset="MA03-1" device="" package3d_urn="urn:adsk.eagle:package:8339/1"/>
+<part name="SV19" library="con-lstb" library_urn="urn:adsk.eagle:library:162" deviceset="MA03-1" device="" package3d_urn="urn:adsk.eagle:package:8339/1"/>
+<part name="SV20" library="con-lstb" library_urn="urn:adsk.eagle:library:162" deviceset="MA03-1" device="" package3d_urn="urn:adsk.eagle:package:8339/1"/>
+<part name="SV21" library="con-lstb" library_urn="urn:adsk.eagle:library:162" deviceset="MA03-1" device="" package3d_urn="urn:adsk.eagle:package:8339/1"/>
+<part name="SV22" library="con-lstb" library_urn="urn:adsk.eagle:library:162" deviceset="MA03-1" device="" package3d_urn="urn:adsk.eagle:package:8339/1"/>
+<part name="SV23" library="con-lstb" library_urn="urn:adsk.eagle:library:162" deviceset="MA03-1" device="" package3d_urn="urn:adsk.eagle:package:8339/1"/>
+<part name="SV24" library="con-lstb" library_urn="urn:adsk.eagle:library:162" deviceset="MA03-1" device="" package3d_urn="urn:adsk.eagle:package:8339/1"/>
+<part name="SV25" library="con-lstb" library_urn="urn:adsk.eagle:library:162" deviceset="MA03-1" device="" package3d_urn="urn:adsk.eagle:package:8339/1"/>
+<part name="SV26" library="con-lstb" library_urn="urn:adsk.eagle:library:162" deviceset="MA03-1" device="" package3d_urn="urn:adsk.eagle:package:8339/1"/>
 </parts>
 <sheets>
@@
 <wire x1="271.78" y1="185.42" x2="220.98" y2="185.42" width="0.1524" layer="97"/>
 <text x="220.98" y="139.7" size="1.778" layer="97">MOTOR CONS</text>
-<text x="325.12" y="154.94" size="1.778" layer="91">TODO:
+<text x="411.226" y="213.36" size="1.778" layer="91">TODO:
 -add serials and values
--add roller and kicker connectors (?)
--add US cons if there's room
--decide which uc, arduino promini (16 sensors) or nano 33 BLE (cooler, allows for 20 sensors)
 -add mux!!!!
 NOTE:
-in brd the spacing of ball sensor is inconsistent in S3, S5, S13</text>
+in brd the spacing of ball sensor is inconsistent in S3, S5, S13
+TODO if i have space:
+-roller/kicker cons
+-US cons</text>
 <text x="50.8" y="223.52" size="2.54" layer="97">M1</text>
 <text x="160.02" y="223.52" size="2.54" layer="97">M2</text>
@@
 <wire x1="520.7" y1="109.22" x2="492.76" y2="109.22" width="0.1524" layer="97"/>
 <text x="492.76" y="76.2" size="1.778" layer="97">BLUETOOTH</text>
-<wire x1="332.74" y1="238.76" x2="332.74" y2="190.5" width="0.1524" layer="97"/>
-<wire x1="332.74" y1="190.5" x2="431.8" y2="190.5" width="0.1524" layer="97"/>
-<wire x1="431.8" y1="190.5" x2="431.8" y2="238.76" width="0.1524" layer="97"/>
-<wire x1="431.8" y1="238.76" x2="332.74" y2="238.76" width="0.1524" layer="97"/>
-<text x="332.74" y="187.96" size="1.778" layer="97">BALL PINHEADERS</text>
+<wire x1="332.74" y1="238.76" x2="332.74" y2="175.26" width="0.1524" layer="97"/>
+<wire x1="332.74" y1="175.26" x2="408.94" y2="175.26" width="0.1524" layer="97"/>
+<wire x1="408.94" y1="175.26" x2="408.94" y2="238.76" width="0.1524" layer="97"/>
+<wire x1="408.94" y1="238.76" x2="332.74" y2="238.76" width="0.1524" layer="97"/>
+<text x="332.74" y="172.72" size="1.778" layer="97">BALL PINHEADERS</text>
 </plain>
 <instances>
@@
 <attribute name="NAME" x="105.41" y="22.098" size="1.778" layer="95" rot="R180"/>
 </instance>
-<instance part="ARDUINO1" gate="G$1" x="149.86" y="78.74" smashed="yes"/>
 <instance part="S1" gate="G$1" x="304.8" y="35.56" smashed="yes">
 <attribute name="NAME" x="302.26" y="45.72" size="1.778" layer="95" rot="R180"/>
@@
 <attribute name="VALUE" x="397.51" y="205.74" size="1.778" layer="96"/>
 <attribute name="NAME" x="397.51" y="219.202" size="1.778" layer="95"/>
+</instance>
+<instance part="SV17" gate="G$1" x="337.82" y="198.12" smashed="yes">
+<attribute name="VALUE" x="336.55" y="190.5" size="1.778" layer="96"/>
+<attribute name="NAME" x="336.55" y="203.962" size="1.778" layer="95"/>
+</instance>
+<instance part="SV18" gate="G$1" x="337.82" y="182.88" smashed="yes">
+<attribute name="VALUE" x="336.55" y="175.26" size="1.778" layer="96"/>
+<attribute name="NAME" x="336.55" y="188.722" size="1.778" layer="95"/>
+</instance>
+<instance part="SV19" gate="G$1" x="353.06" y="198.12" smashed="yes">
+<attribute name="VALUE" x="351.79" y="190.5" size="1.778" layer="96"/>
+<attribute name="NAME" x="351.79" y="203.962" size="1.778" layer="95"/>
+</instance>
+<instance part="SV20" gate="G$1" x="353.06" y="182.88" smashed="yes">
+<attribute name="VALUE" x="351.79" y="175.26" size="1.778" layer="96"/>
+<attribute name="NAME" x="351.79" y="188.722" size="1.778" layer="95"/>
+</instance>
+<instance part="SV21" gate="G$1" x="368.3" y="198.12" smashed="yes">
+<attribute name="VALUE" x="367.03" y="190.5" size="1.778" layer="96"/>
+<attribute name="NAME" x="367.03" y="203.962" size="1.778" layer="95"/>
+</instance>
+<instance part="SV22" gate="G$1" x="368.3" y="182.88" smashed="yes">
+<attribute name="VALUE" x="367.03" y="175.26" size="1.778" layer="96"/>
+<attribute name="NAME" x="367.03" y="188.722" size="1.778" layer="95"/>
+</instance>
+<instance part="SV23" gate="G$1" x="383.54" y="198.12" smashed="yes">
+<attribute name="VALUE" x="382.27" y="190.5" size="1.778" layer="96"/>
+<attribute name="NAME" x="382.27" y="203.962" size="1.778" layer="95"/>
+</instance>
+<instance part="SV24" gate="G$1" x="383.54" y="182.88" smashed="yes">
+<attribute name="VALUE" x="382.27" y="175.26" size="1.778" layer="96"/>
+<attribute name="NAME" x="382.27" y="188.722" size="1.778" layer="95"/>
+</instance>
+<instance part="SV25" gate="G$1" x="398.78" y="198.12" smashed="yes">
+<attribute name="VALUE" x="397.51" y="190.5" size="1.778" layer="96"/>
+<attribute name="NAME" x="397.51" y="203.962" size="1.778" layer="95"/>
+</instance>
+<instance part="SV26" gate="G$1" x="398.78" y="182.88" smashed="yes">
+<attribute name="VALUE" x="397.51" y="175.26" size="1.778" layer="96"/>
+<attribute name="NAME" x="397.51" y="188.722" size="1.778" layer="95"/>
 </instance>
 </instances>
@@
 </segment>
 <segment>
-<pinref part="ARDUINO1" gate="G$1" pin="A2"/>
 <pinref part="SV6" gate="G$1" pin="8"/>
 <wire x1="165.1" y1="76.2" x2="175.26" y2="76.2" width="0.1524" layer="91"/>
@@
 </segment>
 <segment>
-<pinref part="ARDUINO1" gate="G$1" pin="A1"/>
 <pinref part="SV6" gate="G$1" pin="9"/>
 <wire x1="165.1" y1="73.66" x2="175.26" y2="73.66" width="0.1524" layer="91"/>
