File: project/Progetto16sens.brd (EAGLE design)
At the start: 228.6 x 231.1 mm, 127 parts, among them IC1 LMZ14202TZE-ADJ_NOPB, M1 43650-0201, M2 43650-0201, M3 43650-0201, M4 43650-0201, M5 ARDUINO-PRO-MINI

Commit message: help
Parts:
- added J2: 455-1750-1-ND, SparkFun-Connectors:1X03
- J1: device SparkFun-Connectors:1X17 -> SparkFun-Connectors:1X14
- moved LS_4 67.2 mm to (40.6, 52.1)
- moved LS_3 59.7 mm to (40.6, 63.5)
Connections:
- net N$114 renamed BP8
- net N$115 renamed BP9
- net N$116 renamed BP10
- net N$63 renamed BP11
- net N$64 renamed BP12
- net N$70 renamed BP13
- net N$71 renamed BP14
- net N$72 renamed BP15
- net N$73 renamed BP16
- net N$83 renamed BP1
- net N$84 renamed BP2
- net N$87 renamed BP3
- net N$88 renamed BP4
- net N$89 renamed BP5
- net N$90 renamed BP6
- net N$91 renamed BP7
- new net N$114: SV11.1
- new net N$115: SV12.3
- new net N$116: SV12.1
- new net N$117: SV21.3
- new net N$118: SV21.1
- new net N$119: SV13.3
- new net N$120: SV13.1
- new net N$121: SV14.3
- new net N$122: SV14.1
- new net N$123: SV23.3
- new net N$124: SV23.1
- new net N$125: SV15.3
- new net N$126: SV15.1
- new net N$127: SV16.3
- new net N$128: SV16.1
- new net N$129: SV25.3
- new net N$130: SV25.1
- new net N$73: SV7.3
- new net N$83: SV8.1
- new net N$84: SV17.3
- new net N$87: SV17.1
- new net N$88: SV18.3
- new net N$89: SV18.1
- new net N$90: SV19.3
- new net N$91: SV19.1
- net GND: now also SV10.2, SV11.2, SV12.2, SV13.2, SV14.2, SV15.2, SV16.2, SV17.2, SV18.2, SV19.2, SV21.2, SV23.2, SV25.2, SV7.2, SV8.2, SV9.2; no longer M5.J3.1
- net N$110: now also SV10.1; no longer SV3.4, U$1.36/CS
- net N$111: now also SV9.3; no longer SV3.3, U$1.35/TX8
- net N$112: now also SV9.1; no longer SV3.2, U$1.34/RX8
- net N$113: now also SV11.3; no longer SV3.1, U$1.33
- net N$78: now also SV7.1; no longer J1.15, M5.J3.3
- net N$80: now also SV8.3; no longer J1.16, M5.J3.2
- net N$92: now also SV10.3; no longer J1.17
- net PWB_1: now also SV3.1, U$1.33
- net PWB_2: now also SV3.2, U$1.34/RX8
- net PWB_3: now also SV3.3, U$1.35/TX8
- net PWB_4: now also SV3.4, U$1.36/CS

Commit message: started wiring
Parts:
- moved J2 224.4 mm to (86.4, -14.0), turned to 90 degrees
- moved SW_BALL 37.5 mm to (27.9, -33.0)
- moved L_BALL 37.5 mm to (30.5, -24.1)
- moved R_BALL 37.5 mm to (26.7, -24.1)
- moved LS_1 34.7 mm to (55.9, 40.6)
- moved LS_2 34.7 mm to (40.6, 40.6)
- moved C7 14.7 mm to (0.02, -46.0)
- moved C1 14.5 mm to (0.02, -60.5)
- moved C5 2.54 mm to (28.2, -55.9)
- moved C6 2.54 mm to (30.7, -55.9)
- moved C8 2.54 mm to (25.7, -56.4)
- moved SV3 1.27 mm to (15.2, 73.7)
- moved SV6 1.27 mm to (-15.2, 73.7)
- moved SV1 1.27 mm to (-15.3, 35.1)
- moved SV2 1.27 mm to (15.1, 35.1)
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Connections:
- removed net BP1: M5.J7.12, SV4.12
- removed net BP10: M5.J7.1, SV4.1
- removed net BP11: J1.1, M5.J2.2
- removed net BP12: J1.2, M5.J2.1
- removed net BP13: J1.7, M5.J6.5
- removed net BP14: J1.8, M5.J6.6
- removed net BP15: J1.9, M5.J6.7
- removed net BP16: J1.10, M5.J6.8
- removed net BP2: M5.J7.11, SV4.11
- removed net BP3: M5.J7.8, SV4.8
- removed net BP4: M5.J7.7, SV4.7
- removed net BP5: M5.J7.6, SV4.6
- removed net BP6: M5.J7.5, SV4.5
- removed net BP7: M5.J7.4, SV4.4
- removed net BP8: M5.J7.3, SV4.3
- removed net BP9: M5.J7.2, SV4.2
- removed net N$125: SV15.3
- removed net N$126: SV15.1
- removed net N$14: IC1.7, R_ELETT.2
- net +3V3: now also IC1.7, R_ELETT.2
- net B1: now also M5.J7.12, SV4.12
- net B10: now also M5.J7.1, SV4.1
- net B11: now also J1.1, M5.J2.2, SV15.1, SV15.3
- net B12: now also J1.2, M5.J2.1
- net B13: now also J1.7, M5.J6.5
- net B14: now also J1.8, M5.J6.6
- net B15: now also J1.9, M5.J6.7
- net B16: now also J1.10, M5.J6.8
- net B2: now also M5.J7.11, SV4.11
- net B3: now also M5.J7.8, SV4.8
- net B4: now also M5.J7.7, SV4.7
- net B5: now also M5.J7.6, SV4.6
- net B6: now also M5.J7.5, SV4.5
- net B7: now also M5.J7.4, SV4.4
- net B8: now also M5.J7.3, SV4.3
- net B9: now also M5.J7.2, SV4.2
Routing:
- net +12V: track 0.00 -> 59.9 mm, vias 0 -> 2
- net +3V3: track 0.00 -> 25.1 mm
- net N$59: track 0.00 -> 11.9 mm
- net N$55: track 0.00 -> 11.9 mm
- net N$54: track 0.00 -> 11.9 mm
- net N$52: track 0.00 -> 11.9 mm
- net N$82: track 0.00 -> 11.9 mm
- net N$66: track 0.00 -> 11.9 mm
- net N$58: track 0.00 -> 11.9 mm
- net N$57: track 0.00 -> 11.9 mm
- net N$56: track 0.00 -> 11.9 mm
- net N$53: track 0.00 -> 11.9 mm
- net N$50: track 0.00 -> 11.9 mm
- net N$5: track 0.00 -> 11.9 mm
- net N$49: track 0.00 -> 11.9 mm
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
Commit message: started wiring for realllllll
Parts:
- moved DRV3 14.3 mm to (-60.2, 3.81), turned to 270 degrees
- moved DRV2 11.8 mm to (-60.2, 16.5), turned to 90 degrees
- moved M3 4.79 mm to (-61.7, -2.79), flipped to the bottom
- moved M1 4.37 mm to (-71.1, 23.1), flipped to the bottom
- moved C11 4.02 mm to (-47.0, 16.5)
- moved C15 4.02 mm to (-38.1, 16.5)
- moved M2 3.87 mm to (-58.7, 23.1), flipped to the bottom
- moved R17 3.84 mm to (-67.6, -5.33)
- moved R18 3.84 mm to (-65.5, -5.33)
- moved M4 3.81 mm to (-74.2, -2.79), flipped to the bottom
- moved C18 3.59 mm to (-53.1, 14.7)
- moved R5 3.39 mm to (-67.3, 28.2)
- moved R6 3.39 mm to (-65.0, 28.2)
- moved C14 3.34 mm to (-52.8, 5.59), turned to 270 degrees
- moved M4- 2.03 mm to (-71.1, -15.7)
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Connections:
- net M1_OUTA: now also M1.2
- net M1_OUTB: now also M1.1
- net M2_OUTB: no longer M1.1
- net M3_OUTA: no longer M1.2
Routing:
- added copper zone on layer 1, net M1_OUTA
- added copper zone on layer 1, net M1_OUTB
- added copper zone on layer 1, net M2_OUTA
- added copper zone on layer 1, net M2_OUTB
- added copper zone on layer 1, net M3_OUTA
- added copper zone on layer 1, net M3_OUTB
- added copper zone on layer 1, net M4_OUTA
- added copper zone on layer 1, net M4_OUTB
- added copper zone on layer 1, net V-

Commit message: started wiring for realllllll 2
Parts:
- moved L_MOT 8.64 mm to (-13.0, -87.5)
- moved R_MOT 8.64 mm to (-13.0, -87.5)
- moved SW_MOT 8.64 mm to (-13.0, -76.7)
- moved L_ELETT 2.54 mm to (16.5, -87.2)
- moved R_ELETT 2.54 mm to (16.5, -87.0)
- moved SW_ELETT 2.54 mm to (16.5, -76.4)
- moved BAT_CON 2.30 mm to (1.96, -73.0)
- moved L_BAT 2.30 mm to (1.65, -87.5)
- moved R_BAT 2.30 mm to (1.65, -87.5)
Routing:
- net B10: track 0.00 -> 95.7 mm
- net B11: track 0.00 -> 24.8 mm
- net N$86: track 0.00 -> 11.4 mm
- net N$81: track 0.00 -> 11.4 mm
- net N$77: track 0.00 -> 11.4 mm
- net N$76: track 0.00 -> 11.4 mm
- net N$75: track 0.00 -> 11.4 mm
- net N$74: track 0.00 -> 11.4 mm
- net N$65: track 0.00 -> 11.4 mm
- net B16: track 0.00 -> 11.4 mm
- net B15: track 0.00 -> 11.4 mm
- net B14: track 0.00 -> 11.4 mm
- net B13: track 0.00 -> 11.4 mm
- net N$104: track 0.00 -> 7.62 mm
- net B9: track 0.00 -> 7.62 mm
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- added copper zone on layer 1, net GND
- added copper zone on layer 16, net GND
- added copper zone on layer 1, net VBAT
- added copper zone on layer 16, net VBAT

Commit message: greve
Parts:
- moved EXTR_3V3 93.9 mm to (52.1, -59.3), turned to 270 degrees
- moved LS_1 86.9 mm to (-22.9, 77.5)
- moved LS_3 52.7 mm to (-10.2, 77.5)
- moved LS_4 45.8 mm to (2.54, 77.5)
- moved LS_2 44.7 mm to (15.2, 77.5)
- moved BT_CON 20.5 mm to (27.9, 77.5)
- moved SV3 9.25 mm to (17.8, 64.8)
- moved SV6 9.25 mm to (-12.7, 64.8)
- moved U$1 9.25 mm to (1.27, 45.7)
- moved SV1 9.25 mm to (-12.8, 26.3)
- moved SV2 9.25 mm to (17.7, 26.3)
- moved CB4 5.24 mm to (40.5, 80.1)
- moved RB4 5.24 mm to (38.1, 80.1)
Connections:
- removed net VMOT: C1.1, R_MOT.2, SW_MOT.2
- net +12V: now also C1.1, R_MOT.2, SW_MOT.2
Routing:
- net B10: track 95.7 -> 0.66 mm
- net GND: track 6.44 -> 33.0 mm
- added copper zone on layer 1, net +12V

Commit message: aaaaaaaaaaaaaaaaaaaaaaaaaaaaa
Parts:
- added S17, S18, S19: TL32PO, switch:TL3XPO
- moved BALL_MUX 49.1 mm to (43.2, 45.7)
- renumbered SV10 to S_B14, SV11 to S_B8, SV12 to S_B13, SV13 to S_B5, SV14 to S_B12, SV15 to S_B11, SV16 to S_B9, SV17 to S_B10, SV18 to S_B3, SV19 to S_B6, SV21 to S_B2, SV23 to S_B7, SV25 to S_B4, SV7 to S_B1, SV8 to S_B16, SV9 to S_B15
Connections:
- net N$74 renamed SW1
- net N$75 renamed SW2
- net N$76 renamed SW3
- removed net N$110: S_B14.1
- removed net N$111: S_B15.3
- removed net N$112: S_B15.1
- removed net N$113: S_B8.3
- removed net N$114: S_B8.1
- removed net N$115: S_B13.3
- removed net N$116: S_B13.1
- removed net N$117: S_B2.3
- removed net N$118: S_B2.1
- removed net N$119: S_B5.3
- removed net N$120: S_B5.1
- removed net N$121: S_B12.3
- removed net N$122: S_B12.1
- removed net N$123: S_B7.3
- removed net N$124: S_B7.1
- removed net N$127: S_B9.3
- removed net N$128: S_B9.1
- removed net N$129: S_B4.3
- removed net N$130: S_B4.1
- removed net N$57: SV2.4, U$1.29/TX7
- removed net N$58: SV2.3, U$1.30
- removed net N$59: SV2.2, U$1.31
- removed net N$66: SV2.1, U$1.32
- removed net N$73: S_B1.3
- removed net N$78: S_B1.1
- removed net N$80: S_B16.3
- removed net N$83: S_B16.1
- removed net N$84: S_B10.3
- removed net N$87: S_B10.1
- removed net N$88: S_B3.3
- removed net N$89: S_B3.1
- removed net N$90: S_B6.3
- removed net N$91: S_B6.1
- removed net N$92: S_B14.3
- new net A: SV3.4, U$1.36/CS
- new net B: SV3.3, U$1.35/TX8
- new net C: SV3.2, U$1.34/RX8
- new net D: SV3.1, U$1.33
- net B1: now also S_B1.1, S_B1.3
- net B10: now also S_B10.1, S_B10.3
- net B12: now also S_B12.1, S_B12.3
- net B13: now also S_B13.1, S_B13.3
- net B14: now also S_B14.1, S_B14.3
- net B15: now also S_B15.1, S_B15.3
- net B16: now also S_B16.1, S_B16.3
- net B2: now also S_B2.1, S_B2.3
- net B3: now also S_B3.1, S_B3.3
- net B4: now also S_B4.1, S_B4.3
- net B5: now also S_B5.1, S_B5.3
- net B6: now also S_B6.1, S_B6.3
- net B7: now also S_B7.1, S_B7.3
- net B8: now also S_B8.1, S_B8.3
- net B9: now also S_B9.1, S_B9.3
- net PWB_1: now also SV2.4, U$1.29/TX7; no longer SV3.1, U$1.33
- net PWB_2: now also SV2.3, U$1.30; no longer SV3.2, U$1.34/RX8
- net PWB_3: now also SV2.2, U$1.31; no longer SV3.3, U$1.35/TX8
- net PWB_4: now also SV2.1, U$1.32; no longer SV3.4, U$1.36/CS
Routing:
- net PWB_3: track 11.4 -> 47.0 mm, vias 0 -> 2
- net PWB_4: track 11.4 -> 41.7 mm, vias 0 -> 2
- net PWB_1: track 11.4 -> 33.7 mm, vias 0 -> 2
- net PWB_2: track 11.4 -> 30.7 mm, vias 0 -> 2
- net N$58: track 11.9 -> 0.00 mm
- net N$66: track 11.9 -> 0.00 mm
- net N$59: track 11.9 -> 0.00 mm
- net N$57: track 11.9 -> 0.00 mm
- net D: track 0.00 -> 11.4 mm
- net C: track 0.00 -> 11.4 mm
- net B: track 0.00 -> 11.4 mm
- net A: track 0.00 -> 11.4 mm

Commit message: :C
Parts:
- moved S17 102.0 mm to (-41.9, -45.7)
- moved S18 102.0 mm to (-53.3, -45.7)
- moved S19 102.0 mm to (-64.8, -45.7)

Commit message: elaborato checking in two days
Parts:
- removed LS_1, LS_2, LS_3, LS_4: 4P-2.0, OPL_Connector:HW4-2.0
- added LS_E, LS_N, LS_S, LS_W: 4P-2.0, OPL_Connector:HW4-2.0
- moved L_BALL 81.2 mm to (58.4, 52.1)
- moved R_BALL 81.2 mm to (54.6, 52.1)
- moved SW_BALL 81.2 mm to (55.9, 43.2)
- moved BT_CON 79.8 mm to (-50.8, 64.8), turned to 270 degrees
- moved EXTR_3V3 4.84 mm to (47.2, -59.6), turned to 90 degrees
Connections:
- removed net A: SV3.4, U$1.36/CS
- removed net IFE: BT_CON.3
- removed net N$100: SV6.2, U$1.16/A2/RX4/SCL1
- removed net N$101: SV6.1, U$1.15/A1/RX3
- removed net N$102: SV3.12, U$1.14/A0/TX3
- removed net N$104: M5.J7.9, SV4.9
- removed net N$105: SV3.9, U$1.41/A17
- removed net N$106: SV3.8, U$1.40/A16
- removed net N$107: SV3.6, U$1.38/A14/(CS1)
- removed net N$108: SV3.7, U$1.39/A15/(MISO1)
- removed net N$109: SV3.5, U$1.37/CS
- removed net N$13: LS_3.3
- removed net N$15: LS_1.2
- removed net N$16: LS_1.3
- removed net N$17: LS_2.2
- removed net N$18: LS_2.3
- removed net N$19: LS_4.2
- removed net N$20: LS_4.3
- removed net N$37: SV1.11, U$1.0/RX1
- removed net N$38: SV1.10, U$1.1/TX1
- removed net N$39: BT_CON.4
- removed net N$52: SV2.9, U$1.24/A10/TX6/SCL2
- removed net N$53: SV2.8, U$1.25/A11/RX6/SDA2
- removed net N$56: SV2.5, U$1.28/RX7
- removed net N$77: J1.14, M5.J6.12
- removed net N$8: LS_3.2
- removed net N$86: J1.4, M5.J6.2
- removed net N$97: SV6.5, U$1.19/A5/SCL
- removed net N$98: SV6.4, U$1.18/A4/SDA
- removed net N$99: SV6.3, U$1.17/A3/TX4/SDA1
- removed net RXX: U$2.P4
- removed net TXX: U$2.P5
- new net A_RX: M5.J7.11, SV2.4, SV4.11, U$1.29/TX7
- new net A_TX: M5.J7.12, SV2.5, SV4.12, U$1.28/RX7
- new net BT_RX: BT_CON.4, SV1.10, U$1.1/TX1
- new net BT_TX: BT_CON.3, SV1.11, U$1.0/RX1
- new net E_IN: LS_E.2, SV6.2, U$1.16/A2/RX4/SCL1
- new net E_OUT: LS_E.3, SV6.3, U$1.17/A3/TX4/SDA1
- new net N$116: J2.2, M5.J3.2
- new net N$117: J2.3, M5.J3.3
- new net NO: SV2.1, SV2.2, SV2.3, U$1.30, U$1.31, U$1.32
- new net N_IN: LS_N.2, SV6.4, U$1.18/A4/SDA
- new net N_OUT: LS_N.3, SV6.5, U$1.19/A5/SCL
- new net S_IN: LS_S.2, SV3.12, U$1.14/A0/TX3
- new net S_OUT: LS_S.3, SV6.1, U$1.15/A1/RX3
- new net W_IN: LS_W.2, SV3.8, U$1.40/A16
- new net W_OUT: LS_W.3, SV3.9, U$1.41/A17
- net +3V3: now also BALL_MUX.1, LS_E.1, LS_N.1, LS_S.1, LS_W.1; no longer LS_1.1, LS_2.1, LS_3.1, LS_4.1
- net B1: now also J1.1, M5.J2.2; no longer M5.J7.12, SV4.12
- net B11: no longer J1.1, M5.J2.2
- net B12: now also J1.7, M5.J6.5; no longer J1.2, M5.J2.1
- net B13: now also J1.8, M5.J6.6; no longer J1.7, M5.J6.5
- net B14: now also J1.9, M5.J6.7; no longer J1.8, M5.J6.6
- net B15: now also J1.10, M5.J6.8; no longer J1.9, M5.J6.7
- net B16: now also J1.11, M5.J6.9; no longer J1.10, M5.J6.8
- net B2: now also J1.2, M5.J2.1; no longer M5.J7.11, SV4.11
- net GND: now also J1.4, J2.1, LS_E.4, LS_N.4, LS_S.4, LS_W.4, M5.J3.1, M5.J6.2, M5.J7.9, SV4.9; no longer LS_1.4, LS_2.4, LS_3.4, LS_4.4
- net PWB_1: now also SV3.7, U$1.39/A15/(MISO1); no longer SV2.4, U$1.29/TX7
- net PWB_2: now also SV3.6, U$1.38/A14/(CS1); no longer SV2.3, U$1.30
- net PWB_3: now also SV3.5, U$1.37/CS; no longer SV2.2, U$1.31
- net PWB_4: now also SV3.4, U$1.36/CS; no longer SV2.1, U$1.32
- net SCL: now also SV2.9, U$1.24/A10/TX6/SCL2, U$2.P4
- net SDA: now also SV2.8, U$1.25/A11/RX6/SDA2, U$2.P5
- net SW1: now also J1.12, M5.J6.10; no longer J1.11, M5.J6.9
- net SW2: now also J1.13, M5.J6.11; no longer J1.12, M5.J6.10
- net SW3: now also J1.14, M5.J6.12; no longer J1.13, M5.J6.11
Routing:
- net A_RX: track 0.00 -> 51.7 mm, vias 0 -> 1
- net A_TX: track 0.00 -> 50.9 mm, vias 0 -> 1
- net GND: track 33.0 -> 75.2 mm
- net PWB_3: track 47.0 -> 11.4 mm, vias 2 -> 0
- net PWB_4: track 41.7 -> 11.4 mm, vias 2 -> 0
- net B11: track 24.8 -> 0.00 mm
- net NO: track 0.00 -> 23.8 mm
- net PWB_1: track 33.7 -> 11.4 mm, vias 2 -> 0
- net N$116: track 0.00 -> 19.4 mm
- net PWB_2: track 30.7 -> 11.4 mm, vias 2 -> 0
- net B1: track 7.62 -> 24.8 mm
- net N$117: track 0.00 -> 15.9 mm
- net SDA: track 0.00 -> 11.9 mm
- net N$53: track 11.9 -> 0.00 mm
- net SCL: track 0.00 -> 11.9 mm
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Other:
- board text added: "3V3"
- board text added: "GND"
- board text added: "NC"
- board text added: "VIN"
