File: project/Progetto16sens.brd (EAGLE design)
At the start: 228.6 x 231.1 mm, 131 parts, among them IC1 LMZ14202TZE-ADJ_NOPB, J2 455-1750-1-ND, M1 43650-0201, M2 43650-0201, M3 43650-0201, M4 43650-0201, M5 ARDUINO-PRO-MINI

Commit message: elaborato checking in two days
Connections:
- net D renamed SW4
- net N$103 renamed BUZZER
- net N$50 renamed BALL_T
- net N$54 renamed R_DIG
- net N$55 renamed K_DIG
- net N$93 renamed R_PWM
- net N$94 renamed K_PWM
- removed net B: SV3.3, U$1.35/TX8
- removed net C: SV3.2, U$1.34/RX8
- removed net N$40: SV1.9, U$1.2
- removed net N$41: SV1.8, U$1.3
- removed net N$42: SV1.7, U$1.4
- removed net N$43: SV1.6, U$1.5
- removed net N$44: SV1.5, U$1.6
- removed net N$45: SV1.4, U$1.7/RX2
- removed net N$46: SV1.3, U$1.8/TX2
- removed net N$47: SV1.2, U$1.9
- removed net N$48: SV1.1, U$1.10/CS
- removed net N$49: SV2.12, U$1.11/MOSI
- removed net N$5: SV2.10, U$1.3V3
- removed net N$51: SV6.10, U$1.3V3_1
- removed net N$67: SV6.11, U$1.GND_2
- removed net N$82: SV1.12, U$1.GND
- removed net N$95: SV6.7, U$1.21/A7/RX5
- removed net N$96: SV6.6, U$1.20/A6/TX5
- removed net NO: SV2.1, SV2.2, SV2.3, U$1.30, U$1.31, U$1.32
- new net CAM_RX: SV6.6, U$1.20/A6/TX5, U$2.P5
- new net CAM_TX: SV6.7, U$1.21/A7/RX5, U$2.P4
- net +3V3: now also SV2.10, SV6.10, U$1.3V3, U$1.3V3_1
- net BT_RX: now also SV3.3, U$1.35/TX8; no longer SV1.10, U$1.1/TX1
- net BT_TX: now also SV3.2, U$1.34/RX8; no longer SV1.11, U$1.0/RX1
- net M1_INA: now also SV1.11, U$1.0/RX1
- net M1_INB: now also SV1.10, U$1.1/TX1
- net M1_PWM: now also SV1.9, U$1.2
- net M2_INA: now also SV1.8, U$1.3
- net M2_INB: now also SV1.7, U$1.4
- net M2_PWM: now also SV1.6, U$1.5
- net M3_INA: now also SV1.5, U$1.6
- net M3_INB: now also SV1.4, U$1.7/RX2
- net M3_PWM: now also SV1.3, U$1.8/TX2
- net M4_INA: now also SV1.2, U$1.9
- net M4_INB: now also SV1.1, U$1.10/CS
- net M4_PWM: now also SV2.12, U$1.11/MOSI
- net N$69: now also SV1.12, SV6.11, U$1.GND, U$1.GND_2
- net SCL: no longer U$2.P4
- net SDA: no longer U$2.P5
- net SW1: now also SV2.3, U$1.30
- net SW2: now also SV2.2, U$1.31
- net SW3: now also SV2.1, U$1.32
Routing:
- net NO: track 23.8 -> 0.00 mm
- net N$69: track 11.4 -> 34.7 mm
- net +3V3: track 36.8 -> 60.1 mm
- net SW1: track 11.4 -> 23.3 mm
- net N$5: track 11.9 -> 0.00 mm
- net N$82: track 11.9 -> 0.00 mm
- net N$49: track 11.9 -> 0.00 mm
- net N$48: track 11.9 -> 0.00 mm
- net N$47: track 11.9 -> 0.00 mm
- net N$46: track 11.9 -> 0.00 mm
- net N$45: track 11.9 -> 0.00 mm
- net N$44: track 11.9 -> 0.00 mm
- net N$43: track 11.9 -> 0.00 mm
- net N$42: track 11.9 -> 0.00 mm
- net N$41: track 11.9 -> 0.00 mm
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
Commit message: aaaaaaaaaaaaaaaaaaaaa
Parts:
- removed S17, S18, S19: TL32PO, switch:TL3XPO
- added KICK, ROLL: TWIG_2.0, CONNECTER:2.0_1X4
- added LED1, LED2, LED3, L_SW1, L_SW2, L_SW3: (no value), led:CHIPLED_1206
- added PWR1, PWR2: 43650-0201, Molex motori:43650-0200
- added R24, R25, R26: (no value), rcl:R0805
- added R_SW1, R_SW2, R_SW3: (no value), rcl:M0805
- added SG1: F/CM12P, buzzer:F/CM12P
- added SW1, SW2, SW3: TL32PO, switch:TL3XPO
- moved BT_CON 8.03 mm to (-43.2, 62.2)
- moved C13 2.54 mm to (-83.3, 16.5)
- moved C16 2.54 mm to (-77.5, 5.59)
- moved C17 2.54 mm to (-83.3, 5.08)
- moved DRV1 2.54 mm to (-69.8, 16.5)
- moved DRV4 2.54 mm to (-69.8, 3.81)
- moved M1 2.54 mm to (-68.6, 23.1)
- moved M4 2.54 mm to (-71.6, -2.79)
- moved M4+ 2.54 mm to (-68.6, -13.5)
- moved M4- 2.54 mm to (-68.6, -15.7)
- moved R19 2.54 mm to (-68.6, -20.8)
- moved R5 2.54 mm to (-64.8, 28.2)
- moved C11 2.54 mm to (-44.5, 16.5)
- moved C14 2.54 mm to (-50.3, 5.59)
- moved C15 2.54 mm to (-35.6, 16.5)
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Connections:
- net BUZZER renamed BALL_IN
- net SW4 renamed BALL_OUT
- removed net BALL_T: SV2.11, U$1.12/MISO
- new net BUZZ: SG1.+, SV2.11, U$1.12/MISO
- new net LED1: J1.12, M5.J6.10, R26.1
- new net LED2: J1.13, M5.J6.11, R25.1
- new net LED3: J1.14, M5.J6.12, R24.1
- new net N$13: L_SW2.A, R_SW2.1
- new net N$15: R_SW2.2, SW2.3
- new net N$16: L_SW3.A, R_SW3.1
- new net N$17: R_SW3.2, SW3.3
- new net N$18: LED2.A, R25.2
- new net N$19: LED3.A, R24.2
- new net N$20: LED1.A, R26.2
- new net N$5: L_SW1.A, R_SW1.1
- new net N$8: R_SW1.2, SW1.3
- new net VMOT: C1.1, C11.+, C12.1, C13.+, C14.1, C15.+, C16.1, C17.+, C18.1, DRV1.12, DRV1.4, DRV1.5, DRV2.12, DRV2.4, DRV2.5, DRV3.12, DRV3.4, DRV3.5, DRV4.12, DRV4.4, DRV4.5, PWR1.1, PWR2.1, R_MOT.2, SW_MOT.2
- net +12V: no longer C1.1, C11.+, C12.1, C13.+, C14.1, C15.+, C16.1, C17.+, C18.1, DRV1.12, DRV1.4, DRV1.5, DRV2.12, DRV2.4, DRV2.5, DRV3.12, DRV3.4, DRV3.5, DRV4.12, DRV4.4, DRV4.5, R_MOT.2, SW_MOT.2
- net +3V3: now also KICK.1, L_SW1.C, L_SW2.C, L_SW3.C, ROLL.1
- net GND: now also KICK.4, LED1.C, LED2.C, LED3.C, ROLL.4, SG1.-, SW1.1, SW2.1, SW3.1
- net K_DIG: now also KICK.3
- net K_PWM: now also KICK.2
- net R_DIG: now also ROLL.3
- net R_PWM: now also ROLL.2
- net SW1: now also SW1.2; no longer J1.12, M5.J6.10
- net SW2: now also SW2.2; no longer J1.13, M5.J6.11
- net SW3: now also SW3.2; no longer J1.14, M5.J6.12
- net V-: now also PWR1.2, PWR2.2
Routing:
- net BUZZ: track 0.00 -> 11.9 mm
- net BALL_T: track 11.9 -> 0.00 mm
- net SW1: track 23.3 -> 11.9 mm
- net LED3: track 0.00 -> 11.4 mm
- net LED2: track 0.00 -> 11.4 mm
- net LED1: track 0.00 -> 11.4 mm
- net SW3: track 23.3 -> 11.9 mm
- net SW2: track 23.3 -> 11.9 mm
- added copper zone on layer 16, net V-
- added copper zone on layer 1, net VMOT
- removed copper zone on layer 1, net +12V
- removed copper zone on layer 1, net GND

Commit message: first autorouter test....could have gone better
Parts:
- moved C12 0.76 mm to (-77.7, 14.7)
- moved C13 0.76 mm to (-84.1, 16.5)
- moved C16 0.76 mm to (-78.2, 5.59)
- moved C17 0.76 mm to (-84.1, 5.08)
- moved DRV1 0.76 mm to (-70.6, 16.5)
- moved DRV4 0.76 mm to (-70.6, 3.81)
- moved R5 0.51 mm to (-65.3, 28.2)
- moved M1 0.51 mm to (-69.1, 23.1)
- moved M4 0.51 mm to (-72.1, -2.79)
- moved R6 0.51 mm to (-63.0, 28.2)

Commit message: turned in elaborato
Parts:
- moved CB1 9.16 mm to (71.2, 55.1)
- moved RB1 9.16 mm to (71.2, 52.9)
- moved C20 6.35 mm to (45.7, 68.6)
- moved C12 0.76 mm to (-77.0, 14.7)
- moved C13 0.76 mm to (-83.3, 16.5)
- moved C16 0.76 mm to (-77.5, 5.59)
- moved C17 0.76 mm to (-83.3, 5.08)
- moved DRV1 0.76 mm to (-69.8, 16.5)
- moved DRV4 0.76 mm to (-69.8, 3.81)
- moved S_B9 0.57 mm to (-0.25, -96.0)
- moved R5 0.51 mm to (-64.8, 28.2)
- moved M1 0.51 mm to (-68.6, 23.1)
- moved M4 0.51 mm to (-71.6, -2.79)
- moved R6 0.51 mm to (-62.5, 28.2)
- moved S_B5 0.36 mm to (-96.3, -0.51)
Connections:
- removed net N$1: CB2.1, RB2.2, S5.1, S6.3, S7.1, S8.3
- removed net N$2: CB1.1, RB1.2, S1.1, S2.3, S3.1, S4.3
- removed net N$3: CB3.1, RB3.2, S10.3, S11.1, S12.3, S9.1
- removed net N$4: CB4.1, RB4.2, S13.1, S14.3, S15.1, S16.3
- removed net N$69: SV1.12, SV3.10, SV6.11, U$1.GND, U$1.GND_1, U$1.GND_2
- new net PWR_B1: CB1.1, RB1.2, S1.3, S2.3, S3.3, S4.3
- new net PWR_B2: CB2.1, RB2.2, S5.3, S6.3, S7.3, S8.3
- new net PWR_B3: CB3.1, RB3.2, S10.3, S11.3, S12.3, S9.3
- new net PWR_B4: CB4.1, RB4.2, S13.3, S14.3, S15.3, S16.3
- net B1: now also S1.1; no longer S1.3
- net B11: now also S11.1; no longer S11.3
- net B13: now also S13.1; no longer S13.3
- net B15: now also S15.1; no longer S15.3
- net B3: now also S3.1; no longer S3.3
- net B5: now also S5.1; no longer S5.3
- net B7: now also S7.1; no longer S7.3
- net B9: now also S9.1; no longer S9.3
- net GND: now also SV1.12, SV3.10, SV6.11, U$1.GND, U$1.GND_1, U$1.GND_2
Routing:
- net GND: track 75.2 -> 110.0 mm
- net N$69: track 34.7 -> 0.00 mm

Commit message: turned in elaborato
Parts:
- moved M1 0.25 mm to (-68.3, 23.1)
- moved M4 0.25 mm to (-71.4, -2.79)
Routing:
- added copper zone on layer 16, net M1_OUTA
- added copper zone on layer 16, net M1_OUTB
- added copper zone on layer 16, net M2_OUTA
- added copper zone on layer 16, net M2_OUTB
- added copper zone on layer 16, net M3_OUTA
- added copper zone on layer 16, net M3_OUTB
- added copper zone on layer 16, net M4_OUTA
- added copper zone on layer 16, net M4_OUTB
