File: project/Progetto16sens.brd (EAGLE design)
At the start: 228.6 x 231.1 mm, 149 parts, among them IC1 LMZ14202TZE-ADJ_NOPB, J2 455-1750-1-ND, M1 43650-0201, M2 43650-0201, M3 43650-0201, M4 43650-0201, M5 ARDUINO-PRO-MINI, SW1 TL32PO, SW2 TL32PO, SW3 TL32PO

Commit message: BOARD IS DONE EVEN IF IT HAS SOME ZOZZATE and some drill size drc errors but what can u do nowadays
Parts:
- added C21: (no value), rcl:C1206
- added C22, C23: (no value), rcl:C0805
- added LED4: (no value), led:CHIPLED_1206
- added R4: (no value), rcl:R0805
- moved BALL_TAKE 5.24 mm to (-36.8, 76.2)
- moved RB3 4.58 mm to (48.0, -81.8)
- moved CB3 4.58 mm to (48.0, -84.0)
- moved BT_CON 1.27 mm to (-46.6, 62.7)
- moved R_ELETT 0.58 mm to (17.5, -86.8), turned to 180 degrees
- moved L_ELETT 0.39 mm to (17.5, -86.8), turned to 270 degrees
- moved R_BAT 0.18 mm to (2.41, -86.8)
- moved L_BAT 0.17 mm to (2.41, -86.8), turned to 270 degrees
- moved R_MOT 0.13 mm to (-12.1, -86.8)
- moved L_MOT 0.12 mm to (-12.1, -86.8), turned to 90 degrees
Connections:
- removed net N$65: J1.3, M5.J6.1
- removed net N$68: J1.5, M5.J7.10
- removed net N$85: M5.J6.3, SV4.10
- new net N$4: LED4.A, R4.2
- new net RAW: M5.J6.1
- net +3V3: now also C21.1, C22.1, C23.1
- net GND: now also C21.2, C22.2, C23.2, LED4.C
- net LED4: now also R4.1
Routing:
- net +3V3: track 289.7 -> 739.0 mm, vias 2 -> 9
- net CAM_TX: track 0.00 -> 121.7 mm
- net CAM_RX: track 0.00 -> 121.4 mm
- net BT_RX: track 3.70 -> 86.8 mm, vias 0 -> 2
- net BT_TX: track 5.74 -> 88.2 mm
- net SW3: track 58.9 -> 121.6 mm, vias 1 -> 3
- net GND: track 103.2 -> 161.0 mm
- net SW2: track 60.1 -> 114.2 mm, vias 1 -> 3
- net N_OUT: track 0.00 -> 36.7 mm
- net N_IN: track 0.00 -> 36.4 mm
- net LED4: track 0.00 -> 33.9 mm, vias 0 -> 1
- net VMOT: track 0.00 -> 31.0 mm, vias 0 -> 2
- net W_IN: track 0.00 -> 31.0 mm
- net W_OUT: track 0.00 -> 30.8 mm
- net SW1: track 76.6 -> 106.8 mm, vias 1 -> 3
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Other:
- outline, holes or cut-outs redrawn
- board text added: "BALL_IN"
- board text added: "BALL_OUT"
- board text added: "BUZZER"
- board text added: "Designed by Siria Sannino, be creative c:"
- board text added: "E_IN"
- board text added: "E_OUT"
- board text added: "JLCJLCJLC"
- board text added: "KICKER1"
- board text added: "KICKER2"
- board text added: "M1_INA"
- board text added: "M1_INB"
- board text added: "M1_PWM"
- board text added: "M2_INA"
- board text added: "M2_INB"
- board text added: "M2_PWM"
- board text added: "M3_INA"
- board text added: "M3_INB"
- board text added: "M3_PWM"
- board text added: "M4_INA"
- board text added: "M4_INB"
- board text added: "M4_PWM"
- board text added: "MUX1"
- board text added: "MUX2"
- board text added: "MUX3"
- board text added: "MUX4"
- board text added: "N_IN"
- board text added: "N_OUT"
- board text added: "ROLLER1"
- board text added: "ROLLER2"
- board text added: "RX_ARDU"
- board text added: "RX_BT"
- board text added: "RX_CAM"
- board text added: "SCL"
- board text added: "SDA"
- board text added: "SW1"
- board text added: "SW2"
- board text added: "SW3"
- board text added: "S_IN"
- board text added: "S_OUT"
- board text added: "TX_ARDU"
- board text added: "TX_BT"
- board text added: "TX_CAM"
- board text added: "W_IN"
- board text added: "W_OUT"
