File: project/Progetto16sens.sch (EAGLE design)
At the start: 127 parts, among them IC1 LMZ14202TZE-ADJ_NOPB, M1 43650-0201, M2 43650-0201, M3 43650-0201, M4 43650-0201, M5 ARDUINO-PRO-MINI

Commit message: help
Parts:
- added J2: 455-1750-1-ND, SparkFun-Connectors:CONN_03
- J1: device SparkFun-Connectors:CONN_17 -> SparkFun-Connectors:CONN_14
Connections:
- net N$114 renamed BP8
- net N$115 renamed BP9
- net N$116 renamed BP10
- net N$63 renamed BP11
- net N$64 renamed BP12
- net N$70 renamed BP13
- net N$71 renamed BP14
- net N$72 renamed BP15
- net N$73 renamed BP16
- net N$83 renamed BP1
- net N$84 renamed BP2
- net N$87 renamed BP3
- net N$88 renamed BP4
- net N$89 renamed BP5
- net N$90 renamed BP6
- net N$91 renamed BP7
- new net N$114: SV11.1
- new net N$115: SV12.3
- new net N$116: SV12.1
- new net N$117: SV21.3
- new net N$118: SV21.1
- new net N$119: SV13.3
- new net N$120: SV13.1
- new net N$121: SV14.3
- new net N$122: SV14.1
- new net N$123: SV23.3
- new net N$124: SV23.1
- new net N$125: SV15.3
- new net N$126: SV15.1
- new net N$127: SV16.3
- new net N$128: SV16.1
- new net N$129: SV25.3
- new net N$130: SV25.1
- new net N$73: SV7.3
- new net N$83: SV8.1
- new net N$84: SV17.3
- new net N$87: SV17.1
- new net N$88: SV18.3
- new net N$89: SV18.1
- new net N$90: SV19.3
- new net N$91: SV19.1
- net GND: now also SV10.2, SV11.2, SV12.2, SV13.2, SV14.2, SV15.2, SV16.2, SV17.2, SV18.2, SV19.2, SV21.2, SV23.2, SV25.2, SV7.2, SV8.2, SV9.2; no longer M5.GND.3
- net N$110: now also SV10.1; no longer SV3.4, U$1.36/CS
- net N$111: now also SV9.3; no longer SV3.3, U$1.35/TX8
- net N$112: now also SV9.1; no longer SV3.2, U$1.34/RX8
- net N$113: now also SV11.3; no longer SV3.1, U$1.33
- net N$78: now also SV7.1; no longer J1.15, M5.A7
- net N$80: now also SV8.3; no longer J1.16, M5.A6
- net N$92: now also SV10.3; no longer J1.17
- net PWB_1: now also SV3.1, U$1.33
- net PWB_2: now also SV3.2, U$1.34/RX8
- net PWB_3: now also SV3.3, U$1.35/TX8
- net PWB_4: now also SV3.4, U$1.36/CS
Other:
- note added: "TODO: -add serials and values TODO if i have space: -roller/kicker cons -US cons"
- note removed: "TODO: -add serials and values NOTE: in brd the spacing of ball sensor is inconsistent in S3, S5, S13 TODO if i have space: -roller/kicker cons -US cons"
- moved on the sheet: SV10, SV11, SV12, SV13, SV14, SV15, SV16, SV17, SV18, SV19, SV21, SV23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

Commit message: started wiring
Connections:
- removed net BP1: M5.D1/TX, SV4.12
- removed net BP10: M5.D9, SV4.1
- removed net BP11: J1.1, M5.A5
- removed net BP12: J1.2, M5.A4
- removed net BP13: J1.7, M5.A3
- removed net BP14: J1.8, M5.A2
- removed net BP15: J1.9, M5.A1
- removed net BP16: J1.10, M5.A0
- removed net BP2: M5.D0/RX, SV4.11
- removed net BP3: M5.D2, SV4.8
- removed net BP4: M5.D3, SV4.7
- removed net BP5: M5.D4, SV4.6
- removed net BP6: M5.D5, SV4.5
- removed net BP7: M5.D6, SV4.4
- removed net BP8: M5.D7, SV4.3
- removed net BP9: M5.D8, SV4.2
- removed net N$125: SV15.3
- removed net N$126: SV15.1
- removed net N$14: IC1.VOUT, R_ELETT.2
- net +3V3: now also IC1.VOUT, R_ELETT.2
- net B1: now also M5.D1/TX, SV4.12
- net B10: now also M5.D9, SV4.1
- net B11: now also J1.1, M5.A5, SV15.1, SV15.3
- net B12: now also J1.2, M5.A4
- net B13: now also J1.7, M5.A3
- net B14: now also J1.8, M5.A2
- net B15: now also J1.9, M5.A1
- net B16: now also J1.10, M5.A0
- net B2: now also M5.D0/RX, SV4.11
- net B3: now also M5.D2, SV4.8
- net B4: now also M5.D3, SV4.7
- net B5: now also M5.D4, SV4.6
- net B6: now also M5.D5, SV4.5
- net B7: now also M5.D6, SV4.4
- net B8: now also M5.D7, SV4.3
- net B9: now also M5.D8, SV4.2

Commit message: started wiring for realllllll
Connections:
- net M1_OUTA: now also M1.2
- net M1_OUTB: now also M1.1
- net M2_OUTB: no longer M1.1
- net M3_OUTA: no longer M1.2
Changed lines of the file:
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@@
 <setting verticaltext="up"/>
 </settings>
-<grid distance="0.1" unitdist="inch" unit="inch" style="lines" multiple="1" display="no" altdistance="0.05" altunitdist="inch" altunit="inch"/>
+<grid distance="0.1" unitdist="inch" unit="inch" style="lines" multiple="1" display="no" altdistance="0.01" altunitdist="inch" altunit="inch"/>
 <layers>
 <layer number="1" name="Top" color="4" fill="1" visible="no" active="no"/>
@@
 </segment>
 <segment>
-<pinref part="M1" gate="G$1" pin="1"/>
-<wire x1="223.52" y1="177.8" x2="236.22" y2="177.8" width="0.1524" layer="91"/>
-<label x="223.52" y="177.8" size="1.778" layer="95"/>
-</segment>
-<segment>
 <pinref part="DRV2" gate="G$1" pin="OUT_B_1"/>
 <wire x1="144.78" y1="203.2" x2="129.54" y2="203.2" width="0.1524" layer="91"/>
@@
 <wire x1="256.54" y1="157.48" x2="269.24" y2="157.48" width="0.1524" layer="91"/>
 <label x="259.08" y="157.48" size="1.778" layer="95"/>
-</segment>
-<segment>
-<pinref part="M1" gate="G$1" pin="2"/>
-<wire x1="256.54" y1="177.8" x2="269.24" y2="177.8" width="0.1524" layer="91"/>
-<label x="259.08" y="177.8" size="1.778" layer="95"/>
 </segment>
 <segment>
@@
 <label x="78.74" y="215.9" size="1.778" layer="95"/>
 </segment>
+<segment>
+<pinref part="M1" gate="G$1" pin="2"/>
+<wire x1="256.54" y1="177.8" x2="269.24" y2="177.8" width="0.1524" layer="91"/>
+<label x="259.08" y="177.8" size="1.778" layer="95"/>
+</segment>
 </net>
 <net name="M1_OUTB" class="0">
@@
 <label x="78.74" y="200.66" size="1.778" layer="95"/>
 </segment>
-</net>
+<segment>
+<pinref part="M1" gate="G$1" pin="1"/>
+<wire x1="223.52" y1="177.8" x2="236.22" y2="177.8" width="0.1524" layer="91"/>
+<label x="223.52" y="177.8" size="1.778" layer="95"/>
+</segment>
+</net>

Commit message: greve
Connections:
- removed net VMOT: C1.+, R_MOT.2, SW_MOT.P
- net +12V: now also C1.+, R_MOT.2, SW_MOT.P
Changed lines of the file:
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@@
-</segment>
-</net>
-<net name="VMOT" class="0">
-<segment>
-<pinref part="SW_MOT" gate="1" pin="P"/>
-<wire x1="261.62" y1="101.6" x2="264.16" y2="101.6" width="0.1524" layer="91"/>
-<pinref part="R_MOT" gate="G$1" pin="2"/>
-<wire x1="264.16" y1="101.6" x2="271.78" y2="101.6" width="0.1524" layer="91"/>
-<wire x1="271.78" y1="101.6" x2="275.59" y2="101.6" width="0.1524" layer="91"/>
-<wire x1="264.16" y1="104.14" x2="264.16" y2="101.6" width="0.1524" layer="91"/>
-<junction x="264.16" y="101.6"/>
-<pinref part="C1" gate="G$1" pin="+"/>
-<wire x1="271.78" y1="104.14" x2="271.78" y2="101.6" width="0.1524" layer="91"/>
-<junction x="271.78" y="101.6"/>
-<label x="275.59" y="101.6" size="1.778" layer="95" xref="yes"/>
 </segment>
 </net>
@@
 </net>
 <net name="+12V" class="0">
-<segment>
-<pinref part="SW_ELETT" gate="1" pin="P"/>
-<wire x1="261.62" y1="124.46" x2="276.86" y2="124.46" width="0.1524" layer="91"/>
-<label x="276.86" y="124.46" size="1.778" layer="95" xref="yes"/>
-</segment>
 <segment>
 <pinref part="IC1" gate="G$1" pin="VIN"/>
@@
 <junction x="204.47" y="161.29"/>
 </segment>
+<segment>
+<pinref part="SW_MOT" gate="1" pin="P"/>
+<wire x1="261.62" y1="101.6" x2="264.16" y2="101.6" width="0.1524" layer="91"/>
+<pinref part="R_MOT" gate="G$1" pin="2"/>
+<wire x1="264.16" y1="101.6" x2="271.78" y2="101.6" width="0.1524" layer="91"/>
+<wire x1="264.16" y1="104.14" x2="264.16" y2="101.6" width="0.1524" layer="91"/>
+<junction x="264.16" y="101.6"/>
+<pinref part="C1" gate="G$1" pin="+"/>
+<wire x1="271.78" y1="104.14" x2="271.78" y2="101.6" width="0.1524" layer="91"/>
+<junction x="271.78" y="101.6"/>
+<pinref part="SW_ELETT" gate="1" pin="P"/>
+<wire x1="261.62" y1="124.46" x2="277.876" y2="124.46" width="0.1524" layer="91"/>
+<label x="277.876" y="124.46" size="1.778" layer="95" xref="yes"/>
+<wire x1="271.78" y1="101.6" x2="277.876" y2="101.6" width="0.1524" layer="91"/>
+<wire x1="277.876" y1="101.6" x2="277.876" y2="124.46" width="0.1524" layer="91"/>
+</segment>
 </net>
 <net name="N$6" class="0">
@@
 <pinref part="U$1" gate="G$1" pin="34/RX8"/>
 <pinref part="SV3" gate="G$1" pin="2"/>
-<wire x1="83.82" y1="30.48" x2="95.25" y2="30.48" width="0.1524" layer="91"/>
+<wire x1="76.2" y1="30.48" x2="95.25" y2="30.48" width="0.1524" layer="91"/>
 <label x="83.82" y="30.48" size="1.778" layer="95"/>
 </segment>
@@
 <pinref part="U$1" gate="G$1" pin="33"/>
 <pinref part="SV3" gate="G$1" pin="1"/>
-<wire x1="83.82" y1="27.94" x2="95.25" y2="27.94" width="0.1524" layer="91"/>
+<wire x1="76.2" y1="27.94" x2="95.25" y2="27.94" width="0.1524" layer="91"/>
 <label x="83.82" y="27.94" size="1.778" layer="95"/>
 </segment>
@@
 <pinref part="U$1" gate="G$1" pin="35/TX8"/>
 <pinref part="SV3" gate="G$1" pin="3"/>
-<wire x1="83.82" y1="33.02" x2="95.25" y2="33.02" width="0.1524" layer="91"/>
+<wire x1="76.2" y1="33.02" x2="95.25" y2="33.02" width="0.1524" layer="91"/>
 <label x="83.82" y="33.02" size="1.778" layer="95"/>
 </segment>
@@
 <pinref part="U$1" gate="G$1" pin="36/CS"/>
 <pinref part="SV3" gate="G$1" pin="4"/>
-<wire x1="83.82" y1="35.56" x2="95.25" y2="35.56" width="0.1524" layer="91"/>
+<wire x1="76.2" y1="35.56" x2="95.25" y2="35.56" width="0.1524" layer="91"/>
 <label x="83.82" y="35.56" size="1.778" layer="95"/>
 </segment>
@@
 <pinref part="U$1" gate="G$1" pin="VIN"/>
 <pinref part="SV6" gate="G$1" pin="12"/>
-<wire x1="83.82" y1="86.36" x2="95.25" y2="86.36" width="0.1524" layer="91"/>
+<wire x1="76.2" y1="86.36" x2="95.25" y2="86.36" width="0.1524" layer="91"/>
 </segment>
 </net>
@@
 <pinref part="U$1" gate="G$1" pin="23/A9"/>
 <pinref part="SV6" gate="G$1" pin="9"/>
-<wire x1="83.82" y1="78.74" x2="95.25" y2="78.74" width="0.1524" layer="91"/>
+<wire x1="76.2" y1="78.74" x2="95.25" y2="78.74" width="0.1524" layer="91"/>
 </segment>
 </net>
@@
 <pinref part="U$1" gate="G$1" pin="22/A8"/>
 <pinref part="SV6" gate="G$1" pin="8"/>
-<wire x1="83.82" y1="76.2" x2="95.25" y2="76.2" width="0.1524" layer="91"/>
+<wire x1="76.2" y1="76.2" x2="95.25" y2="76.2" width="0.1524" layer="91"/>
 </segment>
 </net>
@@
 <pinref part="U$1" gate="G$1" pin="21/A7/RX5"/>
 <pinref part="SV6" gate="G$1" pin="7"/>
-<wire x1="83.82" y1="73.66" x2="95.25" y2="73.66" width="0.1524" layer="91"/>
+<wire x1="76.2" y1="73.66" x2="95.25" y2="73.66" width="0.1524" layer="91"/>
 </segment>
 </net>
@@
 <segment>
 <pinref part="U$1" gate="G$1" pin="20/A6/TX5"/>
-<wire x1="83.82" y1="71.12" x2="95.25" y2="71.12" width="0.1524" layer="91"/>
+<wire x1="76.2" y1="71.12" x2="95.25" y2="71.12" width="0.1524" layer="91"/>
 <pinref part="SV6" gate="G$1" pin="6"/>
 </segment>
@@
 <pinref part="U$1" gate="G$1" pin="19/A5/SCL"/>
 <pinref part="SV6" gate="G$1" pin="5"/>
-<wire x1="83.82" y1="68.58" x2="95.25" y2="68.58" width="0.1524" layer="91"/>
+<wire x1="76.2" y1="68.58" x2="95.25" y2="68.58" width="0.1524" layer="91"/>
 </segment>
 </net>
@@
 <pinref part="U$1" gate="G$1" pin="18/A4/SDA"/>
 <pinref part="SV6" gate="G$1" pin="4"/>
-<wire x1="83.82" y1="66.04" x2="95.25" y2="66.04" width="0.1524" layer="91"/>
+<wire x1="76.2" y1="66.04" x2="95.25" y2="66.04" width="0.1524" layer="91"/>
 </segment>
 </net>
@@
 <pinref part="U$1" gate="G$1" pin="17/A3/TX4/SDA1"/>
 <pinref part="SV6" gate="G$1" pin="3"/>
-<wire x1="83.82" y1="63.5" x2="95.25" y2="63.5" width="0.1524" layer="91"/>
+<wire x1="76.2" y1="63.5" x2="95.25" y2="63.5" width="0.1524" layer="91"/>
 </segment>
 </net>
@@
 <pinref part="U$1" gate="G$1" pin="16/A2/RX4/SCL1"/>
 <pinref part="SV6" gate="G$1" pin="2"/>
-<wire x1="83.82" y1="60.96" x2="95.25" y2="60.96" width="0.1524" layer="91"/>
+<wire x1="76.2" y1="60.96" x2="95.25" y2="60.96" width="0.1524" layer="91"/>
 </segment>
 </net>
@@
 <pinref part="U$1" gate="G$1" pin="15/A1/TX3"/>
 <pinref part="SV6" gate="G$1" pin="1"/>
-<wire x1="83.82" y1="58.42" x2="95.25" y2="58.42" width="0.1524" layer="91"/>
+<wire x1="76.2" y1="58.42" x2="95.25" y2="58.42" width="0.1524" layer="91"/>
 </segment>
 </net>
@@
 <pinref part="U$1" gate="G$1" pin="14/A0/TX3"/>
 <pinref part="SV3" gate="G$1" pin="12"/>
-<wire x1="83.82" y1="55.88" x2="95.25" y2="55.88" width="0.1524" layer="91"/>
+<wire x1="76.2" y1="55.88" x2="95.25" y2="55.88" width="0.1524" layer="91"/>
 </segment>
 </net>
@@
 <pinref part="U$1" gate="G$1" pin="13(LED)/SCK"/>
 <pinref part="SV3" gate="G$1" pin="11"/>
-<wire x1="83.82" y1="53.34" x2="95.25" y2="53.34" width="0.1524" layer="91"/>
+<wire x1="76.2" y1="53.34" x2="95.25" y2="53.34" width="0.1524" layer="91"/>
 </segment>
 </net>
@@
 <pinref part="U$1" gate="G$1" pin="41/A17"/>
 <pinref part="SV3" gate="G$1" pin="9"/>
-<wire x1="83.82" y1="48.26" x2="95.25" y2="48.26" width="0.1524" layer="91"/>
+<wire x1="76.2" y1="48.26" x2="95.25" y2="48.26" width="0.1524" layer="91"/>
 </segment>
 </net>
@@
 <pinref part="U$1" gate="G$1" pin="40/A16"/>
 <pinref part="SV3" gate="G$1" pin="8"/>
-<wire x1="83.82" y1="45.72" x2="95.25" y2="45.72" width="0.1524" layer="91"/>
+<wire x1="76.2" y1="45.72" x2="95.25" y2="45.72" width="0.1524" layer="91"/>
 </segment>
 </net>
@@
 <pinref part="U$1" gate="G$1" pin="38/A14/(CS1)"/>
 <pinref part="SV3" gate="G$1" pin="6"/>
-<wire x1="83.82" y1="40.64" x2="95.25" y2="40.64" width="0.1524" layer="91"/>
+<wire x1="76.2" y1="40.64" x2="95.25" y2="40.64" width="0.1524" layer="91"/>
 </segment>
 </net>
@@
 <segment>
 <pinref part="U$1" gate="G$1" pin="39/A15/(MISO1)"/>
-<wire x1="83.82" y1="43.18" x2="95.25" y2="43.18" width="0.1524" layer="91"/>
+<wire x1="76.2" y1="43.18" x2="95.25" y2="43.18" width="0.1524" layer="91"/>
 <pinref part="SV3" gate="G$1" pin="7"/>
 </segment>
@@
 <segment>
 <pinref part="U$1" gate="G$1" pin="37/CS"/>
-<wire x1="83.82" y1="38.1" x2="95.25" y2="38.1" width="0.1524" layer="91"/>
+<wire x1="76.2" y1="38.1" x2="95.25" y2="38.1" width="0.1524" layer="91"/>
 <pinref part="SV3" gate="G$1" pin="5"/>
 </segment>
@@
 <pinref part="U$1" gate="G$1" pin="3V3_1"/>
 <pinref part="SV6" gate="G$1" pin="10"/>
-<wire x1="83.82" y1="81.28" x2="95.25" y2="81.28" width="0.1524" layer="91"/>
+<wire x1="76.2" y1="81.28" x2="95.25" y2="81.28" width="0.1524" layer="91"/>
 </segment>
 </net>
@@
 <pinref part="SV6" gate="G$1" pin="11"/>
 <pinref part="U$1" gate="G$1" pin="GND_2"/>
-<wire x1="83.82" y1="83.82" x2="95.25" y2="83.82" width="0.1524" layer="91"/>
+<wire x1="76.2" y1="83.82" x2="95.25" y2="83.82" width="0.1524" layer="91"/>
 </segment>
 </net>
@@
 <pinref part="SV3" gate="G$1" pin="10"/>
 <pinref part="U$1" gate="G$1" pin="GND_1"/>
-<wire x1="83.82" y1="50.8" x2="95.25" y2="50.8" width="0.1524" layer="91"/>
-</segment>
-</net>
+<wire x1="76.2" y1="50.8" x2="95.25" y2="50.8" width="0.1524" layer="91"/>
+</segment>
+</net>

Commit message: aaaaaaaaaaaaaaaaaaaaaaaaaaaaa
Parts:
- removed SV10, SV11, SV12, SV13, SV14, SV15, SV16, SV18, SV7, SV8, SV9: (no value), con-lstb:MA03-1
- added S17, S18, S19: TL32PO, switch:TL32PO
- added S_B1, S_B10, S_B16, S_B2, S_B3, S_B4, S_B5, S_B6, S_B7, S_B8, S_B9: (no value), con-lstb:MA03-1
- renumbered SV17 to S_B11, SV19 to S_B12, SV21 to S_B13, SV23 to S_B14, SV25 to S_B15
Connections:
- net N$74 renamed SW1
- net N$75 renamed SW2
- net N$76 renamed SW3
- removed net N$110: SV10.1
- removed net N$111: SV9.3
- removed net N$112: SV9.1
- removed net N$113: SV11.3
- removed net N$114: SV11.1
- removed net N$115: SV12.3
- removed net N$116: SV12.1
- removed net N$117: S_B13.3
- removed net N$118: S_B13.1
- removed net N$119: SV13.3
- removed net N$120: SV13.1
- removed net N$121: SV14.3
- removed net N$122: SV14.1
- removed net N$123: S_B14.3
- removed net N$124: S_B14.1
- removed net N$127: SV16.3
- removed net N$128: SV16.1
- removed net N$129: S_B15.3
- removed net N$130: S_B15.1
- removed net N$57: SV2.4, U$1.29/TX7
- removed net N$58: SV2.3, U$1.30
- removed net N$59: SV2.2, U$1.31
- removed net N$66: SV2.1, U$1.32
- removed net N$73: SV7.3
- removed net N$78: SV7.1
- removed net N$80: SV8.3
- removed net N$83: SV8.1
- removed net N$84: S_B11.3
- removed net N$87: S_B11.1
- removed net N$88: SV18.3
- removed net N$89: SV18.1
- removed net N$90: S_B12.3
- removed net N$91: S_B12.1
- removed net N$92: SV10.3
- new net A: SV3.4, U$1.36/CS
- new net B: SV3.3, U$1.35/TX8
- new net C: SV3.2, U$1.34/RX8
- new net D: SV3.1, U$1.33
- net B1: now also S_B1.1, S_B1.3
- net B10: now also S_B10.1, S_B10.3
- net B11: now also S_B11.1, S_B11.3; no longer SV15.1, SV15.3
- net B12: now also S_B12.1, S_B12.3
- net B13: now also S_B13.1, S_B13.3
- net B14: now also S_B14.1, S_B14.3
- net B15: now also S_B15.1, S_B15.3
- net B16: now also S_B16.1, S_B16.3
- net B2: now also S_B2.1, S_B2.3
- net B3: now also S_B3.1, S_B3.3
- net B4: now also S_B4.1, S_B4.3
- net B5: now also S_B5.1, S_B5.3
- net B6: now also S_B6.1, S_B6.3
- net B7: now also S_B7.1, S_B7.3
- net B8: now also S_B8.1, S_B8.3
- net B9: now also S_B9.1, S_B9.3
- net GND: now also S_B1.2, S_B10.2, S_B16.2, S_B2.2, S_B3.2, S_B4.2, S_B5.2, S_B6.2, S_B7.2, S_B8.2, S_B9.2; no longer SV10.2, SV11.2, SV12.2, SV13.2, SV14.2, SV15.2, SV16.2, SV18.2, SV7.2, SV8.2, SV9.2
- net PWB_1: now also SV2.4, U$1.29/TX7; no longer SV3.1, U$1.33
- net PWB_2: now also SV2.3, U$1.30; no longer SV3.2, U$1.34/RX8
- net PWB_3: now also SV2.2, U$1.31; no longer SV3.3, U$1.35/TX8
- net PWB_4: now also SV2.1, U$1.32; no longer SV3.4, U$1.36/CS
Other:
- moved on the sheet: SV1, SV2

Commit message: elaborato checking in two days
Parts:
- renumbered LS_1 to LS_N, LS_2 to LS_E, LS_3 to LS_S, LS_4 to LS_W
Connections:
- removed net A: SV3.4, U$1.36/CS
- removed net IFE: BT_CON.3
- removed net N$100: SV6.2, U$1.16/A2/RX4/SCL1
- removed net N$101: SV6.1, U$1.15/A1/TX3
- removed net N$102: SV3.12, U$1.14/A0/TX3
- removed net N$104: M5.GND.1, SV4.9
- removed net N$105: SV3.9, U$1.41/A17
- removed net N$106: SV3.8, U$1.40/A16
- removed net N$107: SV3.6, U$1.38/A14/(CS1)
- removed net N$108: SV3.7, U$1.39/A15/(MISO1)
- removed net N$109: SV3.5, U$1.37/CS
- removed net N$13: LS_S.3
- removed net N$15: LS_N.2
- removed net N$16: LS_N.3
- removed net N$17: LS_E.2
- removed net N$18: LS_E.3
- removed net N$19: LS_W.2
- removed net N$20: LS_W.3
- removed net N$37: SV1.11, U$1.0/RX1
- removed net N$38: SV1.10, U$1.1/TX1
- removed net N$39: BT_CON.4
- removed net N$52: SV2.9, U$1.24/A10/TX6/SCL2
- removed net N$53: SV2.8, U$1.25/A11/RX6/SDA2
- removed net N$56: SV2.5, U$1.28/RX7
- removed net N$77: J1.14, M5.D10
- removed net N$8: LS_S.2
- removed net N$86: J1.4, M5.GND.2
- removed net N$97: SV6.5, U$1.19/A5/SCL
- removed net N$98: SV6.4, U$1.18/A4/SDA
- removed net N$99: SV6.3, U$1.17/A3/TX4/SDA1
- removed net RXX: U$2.P4
- removed net TXX: U$2.P5
- new net A_RX: M5.D0/RX, SV2.4, SV4.11, U$1.29/TX7
- new net A_TX: M5.D1/TX, SV2.5, SV4.12, U$1.28/RX7
- new net BT_RX: BT_CON.4, SV1.10, U$1.1/TX1
- new net BT_TX: BT_CON.3, SV1.11, U$1.0/RX1
- new net E_IN: LS_E.2, SV6.2, U$1.16/A2/RX4/SCL1
- new net E_OUT: LS_E.3, SV6.3, U$1.17/A3/TX4/SDA1
- new net N$116: J2.2, M5.A6
- new net N$117: J2.3, M5.A7
- new net NO: SV2.1, SV2.2, SV2.3, U$1.30, U$1.31, U$1.32
- new net N_IN: LS_N.2, SV6.4, U$1.18/A4/SDA
- new net N_OUT: LS_N.3, SV6.5, U$1.19/A5/SCL
- new net S_IN: LS_S.2, SV3.12, U$1.14/A0/TX3
- new net S_OUT: LS_S.3, SV6.1, U$1.15/A1/TX3
- new net W_IN: LS_W.2, SV3.8, U$1.40/A16
- new net W_OUT: LS_W.3, SV3.9, U$1.41/A17
- net +3V3: now also BALL_MUX.COMMON_INPUT/OUTPUT
- net B1: now also J1.1, M5.A5; no longer M5.D1/TX, SV4.12
- net B11: no longer J1.1, M5.A5
- net B12: now also J1.7, M5.A3; no longer J1.2, M5.A4
- net B13: now also J1.8, M5.A2; no longer J1.7, M5.A3
- net B14: now also J1.9, M5.A1; no longer J1.8, M5.A2
- net B15: now also J1.10, M5.A0; no longer J1.9, M5.A1
- net B16: now also J1.11, M5.D13; no longer J1.10, M5.A0
- net B2: now also J1.2, M5.A4; no longer M5.D0/RX, SV4.11
- net GND: now also J1.4, J2.1, M5.GND.1, M5.GND.2, M5.GND.3, SV4.9
- net PWB_1: now also SV3.7, U$1.39/A15/(MISO1); no longer SV2.4, U$1.29/TX7
- net PWB_2: now also SV3.6, U$1.38/A14/(CS1); no longer SV2.3, U$1.30
- net PWB_3: now also SV3.5, U$1.37/CS; no longer SV2.2, U$1.31
- net PWB_4: now also SV3.4, U$1.36/CS; no longer SV2.1, U$1.32
- net SCL: now also SV2.9, U$1.24/A10/TX6/SCL2, U$2.P4
- net SDA: now also SV2.8, U$1.25/A11/RX6/SDA2, U$2.P5
- net SW1: now also J1.12, M5.D12; no longer J1.11, M5.D13
- net SW2: now also J1.13, M5.D11; no longer J1.12, M5.D12
- net SW3: now also J1.14, M5.D10; no longer J1.13, M5.D11
Other:
- moved on the sheet: C20

Commit message: elaborato checking in two days
Connections:
- net D renamed SW4
- net N$103 renamed BUZZER
- net N$50 renamed BALL_T
- net N$54 renamed R_DIG
- net N$55 renamed K_DIG
- net N$93 renamed R_PWM
- net N$94 renamed K_PWM
- removed net B: SV3.3, U$1.35/TX8
- removed net C: SV3.2, U$1.34/RX8
- removed net N$40: SV1.9, U$1.2
- removed net N$41: SV1.8, U$1.3
- removed net N$42: SV1.7, U$1.4
- removed net N$43: SV1.6, U$1.5
- removed net N$44: SV1.5, U$1.6
- removed net N$45: SV1.4, U$1.7/RX2
- removed net N$46: SV1.3, U$1.8/TX2
- removed net N$47: SV1.2, U$1.9
- removed net N$48: SV1.1, U$1.10/CS
- removed net N$49: SV2.12, U$1.11/MOSI
- removed net N$5: SV2.10, U$1.3V3
- removed net N$51: SV6.10, U$1.3V3_1
- removed net N$67: SV6.11, U$1.GND_2
- removed net N$82: SV1.12, U$1.GND
- removed net N$95: SV6.7, U$1.21/A7/RX5
- removed net N$96: SV6.6, U$1.20/A6/TX5
- removed net NO: SV2.1, SV2.2, SV2.3, U$1.30, U$1.31, U$1.32
- new net CAM_RX: SV6.6, U$1.20/A6/TX5, U$2.P5
- new net CAM_TX: SV6.7, U$1.21/A7/RX5, U$2.P4
- net +3V3: now also SV2.10, SV6.10, U$1.3V3, U$1.3V3_1
- net BT_RX: now also SV3.3, U$1.35/TX8; no longer SV1.10, U$1.1/TX1
- net BT_TX: now also SV3.2, U$1.34/RX8; no longer SV1.11, U$1.0/RX1
- net M1_INA: now also SV1.11, U$1.0/RX1
- net M1_INB: now also SV1.10, U$1.1/TX1
- net M1_PWM: now also SV1.9, U$1.2
- net M2_INA: now also SV1.8, U$1.3
- net M2_INB: now also SV1.7, U$1.4
- net M2_PWM: now also SV1.6, U$1.5
- net M3_INA: now also SV1.5, U$1.6
- net M3_INB: now also SV1.4, U$1.7/RX2
- net M3_PWM: now also SV1.3, U$1.8/TX2
- net M4_INA: now also SV1.2, U$1.9
- net M4_INB: now also SV1.1, U$1.10/CS
- net M4_PWM: now also SV2.12, U$1.11/MOSI
- net N$69: now also SV1.12, SV6.11, U$1.GND, U$1.GND_2
- net SCL: no longer U$2.P4
- net SDA: no longer U$2.P5
- net SW1: now also SV2.3, U$1.30
- net SW2: now also SV2.2, U$1.31
- net SW3: now also SV2.1, U$1.32
Other:
- moved on the sheet: SV3, SV6
