File: project/Progetto16sens.sch (EAGLE design)
At the start: 131 parts, among them IC1 LMZ14202TZE-ADJ_NOPB, J2 455-1750-1-ND, M1 43650-0201, M2 43650-0201, M3 43650-0201, M4 43650-0201, M5 ARDUINO-PRO-MINI

Commit message: aaaaaaaaaaaaaaaaaaaaa
Parts:
- removed S17, S18, S19: TL32PO, switch:TL32PO
- added KICK, ROLL: TWIG_2.0, CONNECTER:TWIG_2.0
- added LED1, LED2, LED3, L_SW1, L_SW2, L_SW3: (no value), led:LEDCHIPLED_1206
- added PWR1, PWR2: 43650-0201, Molex motori:43650-0201
- added R24, R25, R26: (no value), rcl:R-EU_R0805
- added R_SW1, R_SW2, R_SW3: (no value), rcl:R-EU_M0805
- added SG1: F/CM12P, buzzer:F/CM12P
- added SW1, SW2, SW3: TL32PO, switch:TL32PO
Connections:
- net BUZZER renamed BALL_IN
- net SW4 renamed BALL_OUT
- removed net BALL_T: SV2.11, U$1.12/MISO
- new net BUZZ: SG1.1, SV2.11, U$1.12/MISO
- new net LED1: J1.12, M5.D12, R26.1
- new net LED2: J1.13, M5.D11, R25.1
- new net LED3: J1.14, M5.D10, R24.1
- new net N$13: L_SW2.A, R_SW2.1
- new net N$15: R_SW2.2, SW2.S
- new net N$16: L_SW3.A, R_SW3.1
- new net N$17: R_SW3.2, SW3.S
- new net N$18: LED2.A, R25.2
- new net N$19: LED3.A, R24.2
- new net N$20: LED1.A, R26.2
- new net N$5: L_SW1.A, R_SW1.1
- new net N$8: R_SW1.2, SW1.S
- new net VMOT: C1.+, C11.+, C12.1, C13.+, C14.1, C15.+, C16.1, C17.+, C18.1, DRV1.VCC_1, DRV1.VCC_2, DRV1.VCC_3, DRV2.VCC_1, DRV2.VCC_2, DRV2.VCC_3, DRV3.VCC_1, DRV3.VCC_2, DRV3.VCC_3, DRV4.VCC_1, DRV4.VCC_2, DRV4.VCC_3, PWR1.1, PWR2.1, R_MOT.2, SW_MOT.P
- net +12V: no longer C1.+, C11.+, C12.1, C13.+, C14.1, C15.+, C16.1, C17.+, C18.1, DRV1.VCC_1, DRV1.VCC_2, DRV1.VCC_3, DRV2.VCC_1, DRV2.VCC_2, DRV2.VCC_3, DRV3.VCC_1, DRV3.VCC_2, DRV3.VCC_3, DRV4.VCC_1, DRV4.VCC_2, DRV4.VCC_3, R_MOT.2, SW_MOT.P
- net +3V3: now also KICK.1, L_SW1.C, L_SW2.C, L_SW3.C, ROLL.1
- net GND: now also KICK.4, LED1.C, LED2.C, LED3.C, ROLL.4, SG1.2, SW1.O, SW2.O, SW3.O
- net K_DIG: now also KICK.3
- net K_PWM: now also KICK.2
- net R_DIG: now also ROLL.3
- net R_PWM: now also ROLL.2
- net SW1: now also SW1.P; no longer J1.12, M5.D12
- net SW2: now also SW2.P; no longer J1.13, M5.D11
- net SW3: now also SW3.P; no longer J1.14, M5.D10
- net V-: now also PWR1.2, PWR2.2
Other:
- note added: "*in motors the value is VMOT"
- note added: "BUZZER"
- note added: "KICKER"
- note added: "ROLLER"
- note added: "STATUS_LEDS"
- note added: "SWITCHES"
- note removed: "TODO: -add serials and values TODO if i have space: -roller/kicker cons -US cons"
- moved on the sheet: BT_CON, C20, EXTR_3V3, LS_E, LS_N, LS_S, LS_W, S_B1, S_B10, S_B11, S_B12, S_B13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
