File: project/Old_Files/SchedaRobotica.sch (EAGLE design)
At the start: 1 part

Commit message: a lot of things addedgit add .
Parts:
- added BAT_CON: (no value), SparkFun-Connectors:BATTERY_CONN_DEANS
- added BT_CON, LS_1, LS_2, LS_3, LS_4: 4P-2.0, OPL_Connector:GROVE-CONNECTOR-DIP(4P-2.0)
- added C1, C7: EEV-FK1C152Q, Panasonic 1500uF:EEV-FK1C152Q
- added C10, C5, C6: 100u, rcl:C-EUC1206
- added C11, C13, C15, C17: (no value), rcl:CPOL-EUE
- added C12, C14, C16, C18, CB1, CB2, CB3, CB4, CB5: (no value), rcl:C-EUC0805
- added C19, C20: 1u, rcl:C-EUC0805
- added C2, C3, C8: 100n, rcl:C-EUC0805
- added C4, C9: 22n, rcl:C-EUC0805
- added DRV1, DRV2, DRV3, DRV4: VNH7070ASTR, VNH7070AS:VNH7070ASTR
- added EXTR_3V3, M1, M2, M3, M4: 43650-0201, Molex motori:43650-0201
- added IC1: LMZ14202TZE-ADJ_NOPB, LMZ14202TZE:LMZ14202TZE-ADJ_NOPB
- added L_BAT, L_ELETT, L_MOT, M1+, M1-, M2+, M2-, M3+, M3-, M4+, M4-: (no value), led:LEDCHIPLED_1206
- added R1: 61,9k, rcl:R-EU_M0805
- added R10, R11, R12, R13, R14, R15, R16, R17, R18, R19, R20, R5, R6, R7, R8, R9, RB1, RB2, RB3, RB4, RB5, R_BAT, R_ELETT, R_MOT: (no value), rcl:R-EU_M0805
- added R2: 1,07k, rcl:R-EU_M0805
- added R21, R22: 10k, rcl:R-EU_M0805
- added R3: 3,32k, rcl:R-EU_M0805
- added S1, S10, S11, S12, S13, S14, S15, S16, S17, S18, S19, S2, S20, S3, S4, S5, S6, S7, S8, S9: PNA460XM, adafruit:PNA460XM
- added SV1, SV2, SV3, SV4, SV5: (no value), con-lstb:MA12-1
- added SV10, SV11, SV12, SV13, SV14, SV15, SV16, SV17, SV18, SV19, SV20, SV21, SV22, SV23, SV24, SV25, SV26, SV7, SV8, SV9: (no value), con-lstb:MA03-1
- added SV6: (no value), SparkFun-Connectors:CONN_14LONGPADS
- added SW_ELETT, SW_MOT: (no value), switch_modified:255SB
- added U$2: OPENMV_H7, OpenMV:OPENMV_H7
- added U$3: BNO055_BNO055, IMU:BNO055_BNO055
Connections:
- new net +12V: C11.+, C12.1, C13.+, C14.1, C15.+, C16.1, C17.+, C18.1, C2.1, C3.1, C7.+, DRV1.VCC_1, DRV1.VCC_2, DRV1.VCC_3, DRV2.VCC_1, DRV2.VCC_2, DRV2.VCC_3, DRV3.VCC_1, DRV3.VCC_2, DRV3.VCC_3, DRV4.VCC_1, DRV4.VCC_2, DRV4.VCC_3, IC1.VIN, R1.1, SW_ELETT.P
- new net +3V3: BT_CON.1, C10.1, C19.1, C20.1, C5.1, C6.1, C8.1, C9.2, EXTR_3V3.1, LS_1.1, LS_2.1, LS_3.1, LS_4.1, R21.2, R22.2, R3.1, RB1.1, RB2.1, RB3.1, RB4.1, RB5.1, U$2.3V3, U$3.3V3
- new net B1: S1.VCC, SV2.3, SV6.8, U$1.10-CS/MQSR
- new net B10: S10.OUT
- new net B11: S11.VCC
- new net B12: S12.OUT
- new net B13: S13.VCC
- new net B14: S14.OUT
- new net B15: S15.VCC
- new net B16: S16.OUT
- new net B17: S17.VCC
- new net B18: S18.OUT
- new net B19: S19.VCC
- new net B2: S2.OUT, SV2.4, SV6.9, U$1.11-MOSI/CTX1
- new net B20: S20.OUT
- new net B3: S3.VCC
- new net B4: S4.OUT
- new net B5: S5.VCC
- new net B6: S6.OUT
- new net B7: S7.VCC
- new net B8: S8.OUT
- new net B9: S9.VCC
- new net GND: BAT_CON.-, BT_CON.2, C10.2, C19.2, C2.2, C20.2, C3.2, C4.2, C5.2, C6.2, C7.-, C8.2, CB1.2, CB2.2, CB3.2, CB4.2, CB5.2, EXTR_3V3.2, IC1.GND, IC1.GND_EP, LS_1.4, LS_2.4, LS_3.4, LS_4.4, L_BAT.C, L_ELETT.C, L_MOT.C, R11.2, R15.2, R19.2, R2.1, R7.2, S1.GND, S10.GND, S11.GND, S12.GND, S13.GND, S14.GND, S15.GND, S16.GND, S17.GND, S18.GND, S19.GND, S2.GND, S20.GND, S3.GND, S4.GND, S5.GND, S6.GND, S7.GND, S8.GND, S9.GND, SW_ELETT.S, SW_MOT.S, U$1.GND1, U$1.GND2, U$1.GND3, U$1.GND4, U$1.GND5, U$1.GND6, U$2.GND, U$2.PAD1, U$2.PAD2, U$3.GND
- new net IFE: BT_CON.3
- new net M1_INA: M1+.A, R5.1
- new net M1_INB: M1-.A, R6.1
- new net M1_OUTA: DRV1.OUT_A_1, DRV1.OUT_A_2
- new net M1_OUTB: DRV1.OUT_B_1, DRV1.OUT_B_2
- new net M1_PWM: R8.2
- new net M2_INA: M2+.A, R13.1
- new net M2_INB: M2-.A, R14.1
- new net M2_OUTA: DRV2.OUT_A_1, DRV2.OUT_A_2, M2.2
- new net M2_OUTB: DRV2.OUT_B_1, DRV2.OUT_B_2, M1.1, M2.1
- new net M2_PWM: R16.2
- new net M3_INA: M3+.A, R9.1
- new net M3_INB: M3-.A, R10.1
- new net M3_OUTA: DRV3.OUT_A_1, DRV3.OUT_A_2, M1.2, M3.2
- new net M3_OUTB: DRV3.OUT_B_1, DRV3.OUT_B_2, M3.1
- new net M3_PWM: R12.2
- new net M4_INA: M4+.A, R17.1
- new net M4_INB: M4-.A, R18.1
- new net M4_OUTA: DRV4.OUT_A_1, DRV4.OUT_A_2, M4.2
- new net M4_OUTB: DRV4.OUT_B_1, DRV4.OUT_B_2, M4.1
- new net M4_PWM: R20.2
- new net N$1: CB2.1, RB2.2, S5.OUT, S6.VCC, S7.OUT, S8.VCC
- new net N$10: C9.1, IC1.FB, R2.2, R3.2
- new net N$11: IC1.RON, R1.2
- new net N$12: L_ELETT.A, R_ELETT.1
- new net N$13: LS_3.3
- new net N$14: IC1.VOUT, R_ELETT.2
- new net N$15: LS_1.2
- new net N$16: LS_1.3
- new net N$17: LS_2.2
- new net N$18: LS_2.3
- new net N$19: LS_4.2
- new net N$2: CB1.1, RB1.2, S1.OUT, S2.VCC, S3.OUT, S4.VCC
- new net N$20: LS_4.3
- new net N$21: M1+.C, M1-.C, R7.1
- new net N$22: DRV1.IN_A, R5.2
- new net N$23: DRV1.IN_B, R6.2
- new net N$24: DRV1.PWM, R8.1
- new net N$25: DRV3.IN_A, R9.2
- new net N$26: DRV3.IN_B, R10.2
- new net N$27: M3+.C, M3-.C, R11.1
- new net N$28: DRV3.PWM, R12.1
- new net N$29: DRV2.IN_A, R13.2
- new net N$3: CB3.1, RB3.2, S10.VCC, S11.OUT, S12.VCC, S9.OUT
- new net N$30: DRV2.IN_B, R14.2
- new net N$31: M2+.C, M2-.C, R15.1
- new net N$32: DRV2.PWM, R16.1
- new net N$33: DRV4.IN_A, R17.2
- new net N$34: DRV4.IN_B, R18.2
- new net N$35: M4+.C, M4-.C, R19.1
- new net N$36: DRV4.PWM, R20.1
- new net N$39: BT_CON.4
- new net N$4: CB4.1, RB4.2, S13.OUT, S14.VCC, S15.OUT, S16.VCC
- new net N$5: CB5.1, RB5.2, S17.OUT, S18.VCC, S19.OUT, S20.VCC
- new net N$6: C4.1, IC1.SS
- new net N$7: L_BAT.A, R_BAT.2
- new net N$8: LS_3.2
- new net N$9: L_MOT.A, R_MOT.1
- new net RXX: U$2.P4
- new net SCL: R21.1, U$3.SCL
- new net SDA: R22.1, U$3.SDA
- new net TXX: U$2.P5
- new net V-: C1.-, C11.-, C12.2, C13.-, C14.2, C15.-, C16.2, C17.-, C18.2, DRV1.GND_A_1, DRV1.GND_A_2, DRV1.GND_B_1, DRV1.GND_B_2, DRV2.GND_A_1, DRV2.GND_A_2, DRV2.GND_B_1, DRV2.GND_B_2, DRV3.GND_A_1, DRV3.GND_A_2, DRV3.GND_B_1, DRV3.GND_B_2, DRV4.GND_A_1, DRV4.GND_A_2, DRV4.GND_B_1, DRV4.GND_B_2
- new net VBAT: BAT_CON.+, R_BAT.1, SW_ELETT.O, SW_MOT.O
- new net VMOT: C1.+, R_MOT.2, SW_MOT.P
Other:
- note added: "ARDUINO PROMINI"
- note added: "BALL PINHEADERS"
- note added: "BLUETOOTH"
- note added: "EXTR POWER CON"
- note added: "IMU"
- note added: "LINE SENSORS"
- note added: "M1"
- note added: "M2"
- note added: "M3"
- note added: "M4"
- note added: "MOTOR CONS"
- note added: "MOTOR DRIVERS"
- note added: "OPENMV"
- note added: "POWER SWITCHES"
- note added: "POWERBLOCK1"
- note added: "POWERBLOCK2"
- note added: "POWERBLOCK3"
- note added: "POWERBLOCK4"
- note added: "POWERBLOCK5"
- note added: "SUPPLY"
- note added: "TEENSY 4.1"
- note added: "TODO: -add serials and values -add mux!!!! NOTE: in brd the spacing of ball sensor is inconsistent in S3, S5, S13 TODO if i have space: -roller/kicker cons -US cons"
